File: KiCAD/FlightModule/FlightModule.kicad_pcb (KiCad board)
At the start: 2 copper layers, 0 parts

Commit message: 基板とArduinoの位置の決定
Parts:
- added U1: ARDUINO_MKR_WAN_1310, ARDUINO_MKR_WAN_1310:BOARD_ARDUINO_MKR_WAN_1310, F.Cu at (139.0, 100.0)
Other:
- board outline added: 90 x 70 mm
