File: KiCAD/SensingModule/SensingModule/CanInterface.kicad_sch (KiCad schematic)
At the start: 0 parts

Commit message: 基板とmkrの位置を中原さんのものに合わせました
Parts:
- added C4, C5, C6: 0.1uF, Capacitor_SMD:C_0603_1608Metric_Pad1.08x0.95mm_HandSolder, symbol Device:C_Small
- added C7, C8: 15pF, Capacitor_SMD:C_0603_1608Metric_Pad1.08x0.95mm_HandSolder, symbol Device:C_Small
- added D5, D6: B, LED_SMD:LED_0603_1608Metric_Pad1.05x0.95mm_HandSolder, symbol Device:LED_Small
- added R11: 120R, Resistor_SMD:R_0603_1608Metric_Pad0.98x0.95mm_HandSolder, symbol Device:R_Small
- added R12, R13: 680R, Resistor_SMD:R_0603_1608Metric_Pad0.98x0.95mm_HandSolder, symbol Device:R_Small
- added R14: 10kR, Resistor_SMD:R_0603_1608Metric_Pad0.98x0.95mm_HandSolder, symbol Device:R_Small
- added U3: MCP2562-E-P, Package_DIP:DIP-8_W7.62mm, symbol Interface_CAN_LIN:MCP2562-E-P
- added U4: MCP2515-I/P, Package_DIP:DIP-18_W7.62mm, symbol MCP2515-I_P:MCP2515-I/P
- added Y1: 8MHz, Crystal:Crystal_SMD_HC49-SD, symbol Device:Crystal
Connections:
- new net: R14.2, U4.17 (~RESET)
- new net: D5.2 (A), R12.2
- new net: D6.2 (A), R13.2
- new net +3.3V: C5.2, C6.2, R14.1, U3.5 (Vio), U4.18 (VDD)
- new net +5V: C4.2, U3.3 (VDD)
- new net CAN_H: R11.1, U3.7 (CANH)
- new net CAN_L: R11.2, U3.6 (CANL)
- new net CAN_RECEIVE_STATUS: R12.1
- new net CAN_RX: U3.4 (RXD), U4.2 (RXCAN)
- new net CAN_SEND_STATUS: R13.1
- new net CAN_TX: U3.1 (TXD), U4.1 (TXCAN)
- new net GND: C4.1, C5.1, C6.1, C7.2, C8.2, D5.1 (K), D6.1 (K), U3.2 (VSS), U3.8 (STBY), U4.9 (VSS)
- new net OSC1: C7.1, U4.8 (OSC1), Y1.2
- new net OSC2: C8.1, U4.7 (OSC2), Y1.1
- new net SPI_CS_MCP: U4.16 (~CS)
- new net SPI_MISO: U4.15 (SO)
- new net SPI_MOSI: U4.14 (SI)
- new net SPI_SCLK: U4.13 (SCK)
- no-connect marks 0 -> 7
