File: KiCAD/SensingModule/SensingModule/Power.kicad_sch (KiCad schematic)
At the start: 0 parts

Commit message: 基板とmkrの位置を中原さんのものに合わせました
Parts:
- added C1: 10uF, Capacitor_SMD:C_1206_3216Metric_Pad1.33x1.80mm_HandSolder, symbol Device:C_Small
- added C2: 2.2uF, Capacitor_SMD:C_0603_1608Metric_Pad1.08x0.95mm_HandSolder, symbol Device:C_Small
- added C3: 0.1uF, Capacitor_SMD:C_0603_1608Metric_Pad1.08x0.95mm_HandSolder, symbol Device:C_Small
- added D3: R, LED_SMD:LED_0603_1608Metric_Pad1.05x0.95mm_HandSolder, symbol Device:LED_Small
- added D4: GS1010FL, Diode_SMD:D_SOD-123F, symbol Device:D_Small
- added R10: 2.4kR, Resistor_SMD:R_0603_1608Metric_Pad0.98x0.95mm_HandSolder, symbol Device:R_Small
- added U2: NJM7805SDL1, Package_TO_SOT_SMD:TO-252-2, symbol Regulator_Linear:L7805
Connections:
- new net: D3.2 (A), R10.2
- new net +12V: C1.1, D4.1 (K), R10.1, U2.1 (IN)
- new net +5V: C2.1, C3.1, D4.2 (A), U2.3 (OUT)
- new net GND: C1.2, C2.2, C3.2, D3.1 (K), U2.2 (GND)
