File: KiCAD/SensingModule/SensingModule/SensingModule.kicad_sch (KiCad schematic)
At the start: 14 parts, among them J1 BUS, J2 MONITOR, U1 Arduino MKR WAN 1310

Commit message: 基板の中に納めました
Parts:
- U1: footprint ABX00012:ARDUINO_ABX00012 -> ARDUINO_MKR_WAN_1310:BOARD_ARDUINO_MKR_WAN_1310
Changed lines of the file:
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@@
 			)
 		)
-		(property "Footprint" "ABX00012:ARDUINO_ABX00012"
+		(property "Footprint" "ARDUINO_MKR_WAN_1310:BOARD_ARDUINO_MKR_WAN_1310"
 			(at 187.96 74.93 0)
 			(effects
