File: KiCAD/SensingModule/SensingModule/Peripheral.kicad_sch (KiCad schematic)
At the start: 0 parts

Commit message: 基板とmkrの位置を中原さんのものに合わせました
Parts:
- added J3: TERMISTOR, Hirose_Connector:Hirose_DF1B, symbol Connector_Generic:Conn_01x02
- added R15: 10kR, Resistor_SMD:R_0603_1608Metric_Pad0.98x0.95mm_HandSolder, symbol Device:R_Small
- added U10: BME280, Akizuki_BME280_Module:BME280, symbol Akizuki_BME280_Module:BME280
- added U5, U6, U7, U8: MB85RS2MT, Package_DIP:DIP-8_W7.62mm, symbol Memory_NVRAM:MB85RS2MT
- added U9: BNO055, Akizuki_BNO055_Module:BNO055, symbol Akizuki_BNO055_Module:BNO055
Connections:
- new net +3.3V: R15.1, U10.1 (VDD), U10.3 (SCB), U5.3 (~{WP}), U5.7 (~{HOLD}), U5.8 (VDD), U6.3 (~{WP}), U6.7 (~{HOLD}), U6.8 (VDD), U7.3 (~{WP}), U7.7 (~{HOLD}), U7.8 (VDD), U8.3 (~{WP}), U8.7 (~{HOLD}), U8.8 (VDD), U9.1 (VIN)
- new net GND: J3.1 (Pin_1), U10.2 (GND), U10.5 (SDO), U5.4 (GND), U6.4 (GND), U7.4 (GND), U8.4 (GND), U9.7 (GND)
- new net I2C_SCK: U10.6 (SCK), U9.4 (SCL/R)
- new net I2C_SDA: U10.4 (SDI), U9.3 (SDA/T)
- new net SPI_CS_FRAM0: U5.1 (~{CS})
- new net SPI_CS_FRAM1: U6.1 (~{CS})
- new net SPI_CS_FRAM2: U7.1 (~{CS})
- new net SPI_CS_FRAM3: U8.1 (~{CS})
- new net SPI_MISO: U5.2 (SO), U6.2 (SO), U7.2 (SO), U8.2 (SO)
- new net SPI_MOSI: U5.5 (SI), U6.5 (SI), U7.5 (SI), U8.5 (SI)
- new net SPI_SCLK: U5.6 (SCK), U6.6 (SCK), U7.6 (SCK), U8.6 (SCK)
- new net VREF_THERMISTOR: J3.2 (Pin_2), R15.2
- no-connect marks 0 -> 3

Commit message: コネクタ以外は基板の中に入った
Parts:
- J3: footprint Hirose_Connector:Hirose_DF1B -> TSRP_Connector_Hirose:DF51-2P-2DS
Changed lines of the file:
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@@
 			)
 		)
-		(property "Footprint" "Hirose_Connector:Hirose_DF1B"
+		(property "Footprint" "TSRP_Connector_Hirose:DF51-2P-2DS"
 			(at 105.41 46.99 0)
 			(effects
