File: KiCAD/MKRGPSShield/MKRGPSShield_V4.0.kicad_pcb (KiCad board)
At the start: 2 copper layers, 45.7 x 25 mm, 34 parts, among them IC1 SAM-M8Q, J1 -, J2 -, J3 -, U2 AP2112K-3.3

Commit message: GPSSheildのフットプリントを救出
Parts:
- BATT0: footprint BATT-HOLDER_12MM -> Library:BATT-HOLDER_12MM
- C1, C2, C3, C4, R2, R4: footprint 0402-1005X55N -> Library:0402-1005X55N
- D1, D2: footprint SOT65P210X110-3N -> Library:SOT65P210X110-3N
- FD1, FD2, FD3: footprint FD-1-1.5 -> Library:FD-1-1.5
- FRAME1: footprint FRAME -> Library:FRAME
- IC1: footprint UBLOXLIB_SAM-M8Q -> Library:UBLOXLIB_SAM-M8Q
- J1, J2: footprint 1X14_SMD_TH -> Library:1X14_SMD_TH
- J3: footprint SM05B-SRSS-TB -> Library:SM05B-SRSS-TB
- PPS0: footprint LEDC1608X80N-AK -> Library:LEDC1608X80N-AK
- R1: footprint 0402-1005X55N_3633153 -> Library:0402-1005X55N_3633153
- SJ1, SJ2, SJ5, SJ6, SJ7, SJ8: footprint SJ -> Library:SJ
- U$5, U$6, U$7, U$8: footprint MH_RND_F_2.2MM_NM -> Library:MH_RND_F_2.2MM_NM
- U2: footprint SOT25 -> Library:SOT25
- UNK_HOLE_0: footprint dummyfp0 -> Library:dummyfp0
- UNK_HOLE_1: footprint dummyfp1 -> Library:dummyfp1
- UNK_HOLE_2: footprint dummyfp2 -> Library:dummyfp2
- UNK_HOLE_3: footprint dummyfp3 -> Library:dummyfp3
Changed lines of the file:
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@@
 	(net 18 "N$4")
 	(net 19 "N$2")
-	(footprint "1X14_SMD_TH"
+	(footprint "Library:1X14_SMD_TH"
 		(layer "F.Cu")
 		(at 131.9984 115.1636)
@@
 		(embedded_fonts no)
 	)
-	(footprint "1X14_SMD_TH"
+	(footprint "Library:1X14_SMD_TH"
 		(layer "F.Cu")
 		(at 165.0184 94.8436 180)
@@
 		(embedded_fonts no)
 	)
-	(footprint "0402-1005X55N_3633153"
+	(footprint "Library:0402-1005X55N_3633153"
 		(layer "F.Cu")
 		(at 153.8133 106.8983 -90)
@@
 		(embedded_fonts no)
 	)
-	(footprint "dummyfp2"
+	(footprint "Library:dummyfp2"
 		(layer "F.Cu")
 		(at 169.1136 94.7536)
@@
 		(embedded_fonts no)
 	)
-	(footprint "UBLOXLIB_SAM-M8Q"
+	(footprint "Library:UBLOXLIB_SAM-M8Q"
 		(layer "F.Cu")
 		(at 145.1691 104.9655 90)
@@
 		(embedded_fonts no)
 	)
-	(footprint "MH_RND_F_2.2MM_NM"
+	(footprint "Library:MH_RND_F_2.2MM_NM"
 		(layer "F.Cu")
 		(at 169.1136 115.2536 90)
@@
 		(embedded_fonts no)
 	)
-	(footprint "BATT-HOLDER_12MM"
+	(footprint "Library:BATT-HOLDER_12MM"
 		(layer "F.Cu")
 		(at 161.7447 104.0543 -45)
@@
 		)
 		(property "Value" "BATT-HOLDER_12MM"
-			(at -3 9.500009 -225)
+			(at -3 9.500009 135)
 			(unlocked yes)
 			(layer "F.Fab")
@@
 		(embedded_fonts no)
 	)
-	(footprint "0402-1005X55N"
+	(footprint "Library:0402-1005X55N"
 		(layer "F.Cu")
 		(at 133.8386 104.3036 90)
@@
 		(embedded_fonts no)
 	)
-	(footprint "SOT25"
+	(footprint "Library:SOT25"
 		(layer "F.Cu")
 		(at 129.1438 102.035 90)
@@
 		(embedded_fonts no)
 	)
-	(footprint "FD-1-1.5"
+	(footprint "Library:FD-1-1.5"
 		(layer "F.Cu")
 		(at 127.3136 108.2536)
@@
 		(embedded_fonts no)
 	)
-	(footprint "dummyfp1"
+	(footprint "Library:dummyfp1"
 		(layer "F.Cu")
 		(at 169.1136 115.2536)
@@
 		(embedded_fonts no)
 	)
-	(footprint "FD-1-1.5"
+	(footprint "Library:FD-1-1.5"
 		(layer "F.Cu")
 		(at 151.8136 98.6036 90)
@@
 		(embedded_fonts no)
 	)
-	(footprint "MH_RND_F_2.2MM_NM"
+	(footprint "Library:MH_RND_F_2.2MM_NM"
 		(layer "F.Cu")
 		(at 127.8886 115.2536 90)
@@
 		(embedded_fonts no)
 	)
-	(footprint "0402-1005X55N"
+	(footprint "Library:0402-1005X55N"
 		(layer "F.Cu")
 		(at 127.9886 99.4786 180)
@@
 		(embedded_fonts no)
 	)
-	(footprint "dummyfp0"
+	(footprint "Library:dummyfp0"
 		(layer "F.Cu")
 		(at 127.8886 115.2536)
@@
 		(embedded_fonts no)
 	)
-	(footprint "0402-1005X55N"
+	(footprint "Library:0402-1005X55N"
 		(layer "F.Cu")
 		(at 131.8136 100.5786 -90)
@@
 		(embedded_fonts no)
 	)
-	(footprint "0402-1005X55N"
+	(footprint "Library:0402-1005X55N"
 		(layer "F.Cu")
 		(at 155.746 112.0499 -90)
@@
 		(embedded_fonts no)
 	)
-	(footprint "dummyfp3"
+	(footprint "Library:dummyfp3"
 		(layer "F.Cu")
 		(at 127.8886 94.7536)
@@
 		(embedded_fonts no)
 	)
-	(footprint "0402-1005X55N"
+	(footprint "Library:0402-1005X55N"
 		(layer "F.Cu")
 		(at 136.459 98.2631 180)
@@
 		(embedded_fonts no)
 	)
-	(footprint "MH_RND_F_2.2MM_NM"
+	(footprint "Library:MH_RND_F_2.2MM_NM"
 		(layer "F.Cu")
 		(at 169.1136 94.7536 90)
@@
 		(embedded_fonts no)
 	)
-	(footprint "SM05B-SRSS-TB"
+	(footprint "Library:SM05B-SRSS-TB"
 		(layer "F.Cu")
 		(at 128.3136 108.2536 -90)
@@
 		(embedded_fonts no)
 	)
-	(footprint "MH_RND_F_2.2MM_NM"
+	(footprint "Library:MH_RND_F_2.2MM_NM"
 		(layer "F.Cu")
 		(at 127.8886 94.7536 90)
@@
 		(embedded_fonts no)
 	)
-	(footprint "FRAME"
+	(footprint "Library:FRAME"
 		(layer "F.Cu")
 		(at 125.6386 117.5036)
@@
 		(embedded_fonts no)
 	)
-	(footprint "SOT65P210X110-3N"
+	(footprint "Library:SOT65P210X110-3N"
 		(layer "F.Cu")
 		(at 130.7496 98.1234)
@@
 		(embedded_fonts no)
 	)
-	(footprint "0402-1005X55N"
+	(footprint "Library:0402-1005X55N"
 		(layer "F.Cu")
 		(at 131.6136 105.2786)
@@
 		(embedded_fonts no)
 	)
-	(footprint "FD-1-1.5"
+	(footprint "Library:FD-1-1.5"
 		(layer "F.Cu")
 		(at 138.6215 111.5417 90)
@@
 		(embedded_fonts no)
 	)
-	(footprint "LEDC1608X80N-AK"
+	(footprint "Library:LEDC1608X80N-AK"
 		(layer "F.Cu")
 		(at 154.0481 111.5438 90)
@@
 		(embedded_fonts no)
 	)
-	(footprint "SOT65P210X110-3N"
+	(footprint "Library:SOT65P210X110-3N"
 		(layer "F.Cu")
 		(at 133.8386 100.1536 -90)
@@
 		(embedded_fonts no)
 	)
-	(footprint "SJ"
+	(footprint "Library:SJ"
 		(layer "B.Cu")
 		(at 139.1386 98.0036 -90)
@@
 		)
 		(property "Value" "DNP"
-			(at 0.4001 0 -90)
+			(at 0.4001 0 270)
 			(unlocked yes)
 			(layer "B.Fab")
@@
 		(embedded_fonts no)
 	)
-	(footprint "SJ"
+	(footprint "Library:SJ"
 		(layer "B.Cu")
 		(at 162.4386 98.0036 -90)
@@
 		)
 		(property "Value" "DNP"
-			(at 0.4001 0 -90)
+			(at 0.4001 0 270)
 			(unlocked yes)
 			(layer "B.Fab")
@@
 		(embedded_fonts no)
 	)
-	(footprint "SJ"
+	(footprint "Library:SJ"
 		(layer "B.Cu")
 		(at 141.6886 98.0036 -90)
@@
 		)
 		(property "Value" "DNP"
-			(at 0.4001 0 -90)
+			(at 0.4001 0 270)
 			(unlocked yes)
 			(layer "B.Fab")
@@
 		(embedded_fonts no)
 	)
-	(footprint "SJ"
+	(footprint "Library:SJ"
 		(layer "B.Cu")
 		(at 144.2386 98.0036 -90)
@@
 		)
 		(property "Value" "DNP"
-			(at 0.4001 0 -90)
+			(at 0.4001 0 270)
 			(unlocked yes)
 			(layer "B.Fab")
@@
 		(embedded_fonts no)
 	)
-	(footprint "SJ"
+	(footprint "Library:SJ"
 		(layer "B.Cu")
 		(at 159.9286 98.0091 -90)
@@
 		)
 		(property "Value" "DNP"
-			(at 0.4001 0 -90)
+			(at 0.4001 0 270)
 			(unlocked yes)
 			(layer "B.Fab")
@@
 		(embedded_fonts no)
 	)
-	(footprint "SJ"
+	(footprint "Library:SJ"
 		(layer "B.Cu")
 		(at 165.0386 98.0036 -90)
@@
 		)
 		(property "Value" "DNP"
-			(at 0.4001 0 -90)
+			(at 0.4001 0 270)
 			(unlocked yes)
 			(layer "B.Fab")
