File: KiCAD/SubaruPlate/ServoMotor.kicad_sch (KiCad schematic)
At the start: 1 part, among them J2 B3B-XH-A(LF)(SN)

Commit message: 後は最終確認
Parts:
- J2: now not fitted; now left out of the parts list
Changed lines of the file:
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@@
 		(unit 1)
 		(exclude_from_sim no)
-		(in_bom yes)
-		(on_board yes)
-		(dnp no)
+		(in_bom no)
+		(on_board no)
+		(dnp yes)
 		(property "Reference" "J2"
 			(at 55.88 36.8301 0)
