File: KiCAD/SubaruPlate/Power.kicad_sch (KiCad schematic)
At the start: 1 part

Commit message: 後は最終確認
Parts:
- added C11: 22u, Capacitor_SMD:C_0805_2012Metric_Pad1.18x1.45mm_HandSolder, symbol Device:C
- added C12: 10u, Capacitor_SMD:C_0805_2012Metric_Pad1.18x1.45mm_HandSolder, symbol Device:C
- added C8, C9: 1u, Capacitor_SMD:C_0603_1608Metric_Pad1.08x0.95mm_HandSolder, symbol Device:C
- added MD2: OKL-T_6-W12N-C, TSRP_IC:MURATA_OKL-T-6-W12N-C_0, symbol TSRP_IC:OKL-T_6-W12N-C
- added R10: 1k 0.1%, Resistor_SMD:R_0603_1608Metric_Pad0.98x0.95mm_HandSolder, symbol Device:R
- added R11: 330 0.1%, Resistor_SMD:R_0603_1608Metric_Pad0.98x0.95mm_HandSolder, symbol Device:R
- added R12: 10 0.1%, Resistor_SMD:R_0603_1608Metric_Pad0.98x0.95mm_HandSolder, symbol Device:R
- added R8: 20k, Resistor_SMD:R_0603_1608Metric_Pad0.98x0.95mm_HandSolder, symbol Device:R
- added R9: 100k, Resistor_SMD:R_0603_1608Metric_Pad0.98x0.95mm_HandSolder, symbol Device:R
- added U2: NCV8114BSN330T1G, Package_TO_SOT_SMD:TSOT-23-5, symbol Regulator_Linear:NCV8114BSN330T1G
- PS1: now not fitted; now left out of the parts list
Connections:
- net +12V: now also C11.1, MD2.2 (VIN), R8.1
- net +5V: now also C12.1, C8.1, MD2.4 (VOUT), MD2.5 (SENSE), R9.1, U2.1 (IN), U2.3 (EN)
- net GND: now also C11.2, C12.2, C8.2, C9.2, MD2.1 (~{ON}/OFF_CONTROL), MD2.3 (1_GROUND), MD2.7 (2_GROUND), R12.2, R8.2, U2.2 (GND)
- new net: R10.2, R11.1
- new net: R11.2, R12.1
- new net: MD2.6 (TRIM), R10.1
- new net +3.3V: C9.1, U2.5 (OUT)
- new net P.G._OKL-T/6-W12N-C: MD2.10 (POWER_GOOD_OUT), R9.2
- no-connect marks 0 -> 4
Other:
- note added: "本当は，RT9080-33GJ5"

Commit message: 取付穴位置を変更
Parts:
- added C10: 2200uF, Capacitor_THT:CP_Radial_D18.0mm_P7.50mm, symbol Device:C_Polarized_Small
- added J3: DF51A-2P-2DSA, TSRP_Connector_Hirose:DF51A-2P-2DSA, symbol Connector_Generic:Conn_01x02
- C11: value 22u -> 22uF
- C12: value 10u -> 10uF
- C8, C9: value 1u -> 1uF
- R10: value 1k 0.1% -> 1kR 0.1%
- R11: value 330 0.1% -> 330R 0.1%
- R12: value 10 0.1% -> 10R 0.1%
- R8: value 20k -> 20kR
- R9: value 100k -> 100kR
Connections:
- new net Capacitor IN: C10.1, J3.2 (Pin_2)
- new net Capacitor OUT: C10.2, J3.1 (Pin_1)
Other:
- note added: "Capacitor"

Commit message: ガバーデータ生成
Parts:
- added D1: D, Diode_SMD:D_SMA, symbol Device:D
Connections:
- net +12V: now also D1.2 (A); no longer C11.1, MD2.2 (VIN), R8.1
- new net VIN(12V): C11.1, D1.1 (K), MD2.2 (VIN), R8.1
Changed lines of the file:
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@@
 	)
 	(rectangle
-		(start 95.25 25.4)
+		(start 91.44 25.4)
 		(end 274.32 74.93)
 		(stroke
@@
 	)
 	(rectangle
-		(start 99.06 30.48)
-		(end 109.22 38.1)
+		(start 95.25 30.48)
+		(end 105.41 38.1)
 		(stroke
 			(width 0)
@@
 	(text_box "Switching Regulator"
 		(exclude_from_sim no)
-		(at 95.25 21.59 0)
+		(at 91.44 21.59 0)
 		(size 27.94 3.81)
 		(margins 0.9525 0.9525 0.9525 0.9525)
@@
 	(text_box "From BUS"
 		(exclude_from_sim no)
-		(at 97.79 27.94 0)
+		(at 93.98 27.94 0)
 		(size 12.7 2.54)
 		(margins 0.9525 0.9525 0.9525 0.9525)
@@
 	)
 	(junction
+		(at 144.78 39.37)
+		(diameter 0)
+		(color 0 0 0 0)
+	)
+	(junction
 		(at 36.83 116.84)
+		(diameter 0)
+		(color 0 0 0 0)
+	)
+	(junction
+		(at 116.84 39.37)
 		(diameter 0)
 		(color 0 0 0 0)
@@
 	)
 	(junction
-		(at 116.84 39.37)
-		(diameter 0)
-		(color 0 0 0 0)
-	)
-	(junction
 		(at 251.46 39.37)
 		(diameter 0)
@@
 	(wire
 		(pts
+			(xy 115.57 39.37) (xy 116.84 39.37)
+		)
+		(stroke
+			(width 0)
+			(type default)
+		)
+	)
+	(wire
+		(pts
 			(xy 138.43 130.81) (xy 140.97 130.81)
 		)
@@
 	(wire
 		(pts
+			(xy 144.78 34.29) (xy 144.78 39.37)
+		)
+		(stroke
+			(width 0)
+			(type default)
+		)
+	)
+	(wire
+		(pts
+			(xy 144.78 39.37) (xy 149.86 39.37)
+		)
+		(stroke
+			(width 0)
+			(type default)
+		)
+	)
+	(wire
+		(pts
 			(xy 130.81 130.81) (xy 133.35 130.81)
 		)
@@
 	(wire
 		(pts
-			(xy 129.54 39.37) (xy 149.86 39.37)
+			(xy 129.54 39.37) (xy 144.78 39.37)
 		)
 		(stroke
@@
 	(wire
 		(pts
-			(xy 104.14 39.37) (xy 104.14 38.1)
+			(xy 100.33 39.37) (xy 100.33 38.1)
 		)
 		(stroke
@@
 	(wire
 		(pts
+			(xy 143.51 34.29) (xy 144.78 34.29)
+		)
+		(stroke
+			(width 0)
+			(type default)
+		)
+	)
+	(wire
+		(pts
 			(xy 129.54 49.53) (xy 129.54 50.8)
 		)
@@
 	(wire
 		(pts
+			(xy 100.33 39.37) (xy 107.95 39.37)
+		)
+		(stroke
+			(width 0)
+			(type default)
+		)
+	)
+	(wire
+		(pts
 			(xy 93.98 116.84) (xy 93.98 114.3)
-		)
-		(stroke
-			(width 0)
-			(type default)
-		)
-	)
-	(wire
-		(pts
-			(xy 104.14 39.37) (xy 116.84 39.37)
 		)
 		(stroke
@@
 	(label "Capacitor IN"
 		(at 140.97 120.65 0)
+		(effects
+			(font
+				(size 1.27 1.27)
+			)
+			(justify left bottom)
+		)
+	)
+	(label "VIN(12V)"
+		(at 119.38 39.37 0)
 		(effects
 			(font
@@
 		)
 	)
+	(global_label "VIN(12V)"
+		(shape input)
+		(at 143.51 34.29 180)
+		(fields_autoplaced yes)
+		(effects
+			(font
+				(size 1.27 1.27)
+			)
+			(justify right)
+		)
+		(property "Intersheetrefs" "${INTERSHEET_REFS}"
+			(at 132.2999 34.29 0)
+			(effects
+				(font
+					(size 1.27 1.27)
+				)
+				(justify right)
+				(hide yes)
+			)
+		)
+	)
 	(symbol
 		(lib_id "Device:R")
@@
 	)
 	(symbol
+		(lib_id "Device:D")
+		(at 111.76 39.37 180)
+		(unit 1)
+		(exclude_from_sim no)
+		(in_bom yes)
+		(on_board yes)
+		(dnp no)
+		(fields_autoplaced yes)
+		(property "Reference" "D1"
+			(at 111.76 33.02 0)
+			(effects
+				(font
+					(size 1.27 1.27)
+				)
+			)
+		)
+		(property "Value" "D"
+			(at 111.76 35.56 0)
+			(effects
+				(font
+					(size 1.27 1.27)
+				)
+			)
+		)
+		(property "Footprint" "Diode_SMD:D_SMA"
+			(at 111.76 39.37 0)
+			(effects
+				(font
+					(size 1.27 1.27)
+				)
+				(hide yes)
+			)
+		)
+		(property "Datasheet" "~"
+			(at 111.76 39.37 0)
+			(effects
+				(font
+					(size 1.27 1.27)
+				)
+				(hide yes)
+			)
+		)
+		(property "Description" "Diode"
+			(at 111.76 39.37 0)
+			(effects
+				(font
+					(size 1.27 1.27)
+				)
+				(hide yes)
+			)
+		)
+		(property "Sim.Device" "D"
+			(at 111.76 39.37 0)
+			(effects
+				(font
+					(size 1.27 1.27)
+				)
+				(hide yes)
+			)
+		)
+		(property "Sim.Pins" "1=K 2=A"
+			(at 111.76 39.37 0)
+			(effects
+				(font
+					(size 1.27 1.27)
+				)
+				(hide yes)
+			)
+		)
+		(pin "2"
+		)
+		(pin "1"
+		)
+		(instances
+			(project ""
+				(path "/6c4aa1f5-c08b-4349-85f8-88bb399e711f/5080f980-61f3-43e2-a69d-110d0de0a5b0"
+					(reference "D1")
+					(unit 1)
+				)
+			)
+		)
+	)
+	(symbol
 		(lib_id "power:+12V")
-		(at 104.14 38.1 0)
+		(at 100.33 38.1 0)
 		(unit 1)
 		(exclude_from_sim no)
@@
 		(fields_autoplaced yes)
 		(property "Reference" "#PWR041"
-			(at 104.14 41.91 0)
+			(at 100.33 41.91 0)
 			(effects
 				(font
@@
 		)
 		(property "Value" "+12V"
-			(at 104.14 33.02 0)
+			(at 100.33 33.02 0)
 			(effects
 				(font
@@
 		)
 		(property "Footprint" ""
-			(at 104.14 38.1 0)
+			(at 100.33 38.1 0)
 			(effects
 				(font
@@
 		)
 		(property "Datasheet" ""
-			(at 104.14 38.1 0)
+			(at 100.33 38.1 0)
 			(effects
 				(font
@@
 		)
 		(property "Description" "Power symbol creates a global label with name \"+12V\""
-			(at 104.14 38.1 0)
+			(at 100.33 38.1 0)
 			(effects
 				(font
@@
 			)
 		)
-		(property "Datasheet" "~"
+		(property "Datasheet" "https://akizukidenshi.com/catalog/g/g102723/"
 			(at 135.89 130.81 0)
 			(effects

Commit message: Build-2完成．発注．
Parts:
- added D2: SR54F, Diode_SMD:D_SMA, symbol Device:D
- C11, C12, D1, MD2, R10, R11, R12, R8, R9: now not fitted; now left out of the parts list
- PS1: now fitted; now in the parts list
Connections:
- net +12V: now also D2.2 (A); no longer PS1.1 (+VIN)
- new net 12V: D2.1 (K), PS1.1 (+VIN)
Other:
- moved on the sheet: C10, C8, C9, J3, U2
