File: KiCAD/SubaruPlate/Sensor.kicad_sch (KiCad schematic)
At the start: 6 parts, among them U1 LPS28DFW

Commit message: 取付穴位置を変更
Parts:
- R1, R2, R3: value 10K -> 10kR
Changed lines of the file:
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@@
 			)
 		)
-		(property "Value" "10K"
+		(property "Value" "10kR"
 			(at 107.95 54.6099 0)
 			(effects
@@
 			)
 		)
-		(property "Value" "10K"
+		(property "Value" "10kR"
 			(at 97.79 74.9299 0)
 			(effects
@@
 			)
 		)
-		(property "Value" "10K"
+		(property "Value" "10kR"
 			(at 97.79 54.6099 0)
 			(effects

Commit message: ガバーデータ生成
Parts:
- added C13: 0.1uF, Capacitor_SMD:C_0603_1608Metric_Pad1.08x0.95mm_HandSolder, symbol Device:C
- added C14: 10uF, Capacitor_SMD:C_0603_1608Metric_Pad1.08x0.95mm_HandSolder, symbol Device:C
- added R14, R15, R16: 10kR, Resistor_SMD:R_0603_1608Metric_Pad0.98x0.95mm_HandSolder, symbol Device:R
- added U6: LPS28DFW, TSRP_IC:CCLGA-7L, symbol TSRP_IC:LPS28DFW
Connections:
- net +3.3V: now also C13.1, C14.1, R14.1, R16.1, U6.6 (VDD)
- net GND: now also C13.2, C14.2, R15.2, U6.5 (GND), U6.7 (LID)
- net I2C_SCL: now also R16.2, U6.3 (SCL)
- net I2C_SDA: now also R14.2, U6.1 (SDA)
- new net: R15.1, U6.2 (SA0)
- no-connect marks 1 -> 2
Other:
- moved on the sheet: C1, C2, R1, R2, R3, U1

Commit message: Build-2完成．発注．
Parts:
- removed R15: 10kR, Resistor_SMD:R_0603_1608Metric_Pad0.98x0.95mm_HandSolder, symbol Device:R
- added J1: Wire_Soldering, Connector_PinHeader_1.27mm:PinHeader_1x04_P1.27mm_Vertical, symbol Connector_Generic:Conn_01x04
Connections:
- net +3.3V: now also U6.2 (SA0), J1.2 (Pin_2)
- net GND: now also J1.1 (Pin_1)
- net I2C_SCL: now also J1.4 (Pin_4)
- net I2C_SDA: now also J1.3 (Pin_3)
Other:
- note added: "I2C Address: 0x5C"
- note added: "I2C Address: 0x5D"
