File: KiCAD/PowerModule/PowerModule.kicad_pcb (KiCad board)
At the start: 2 copper layers, 90 x 70 mm, 47 parts, among them J2 DF1B-2S-2.5R, J3 DF1B-2S-2.5R, J4 DF1B-2S-2.5R, J5 DF11-8DP-2DS, J6 DF1B-2S-2.5R, J7 DF11-8DP-2DS, J8 DF51-2P-2DS, Q1 AO3401A, Q2 AO3401A, U1 INA219BxDCN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

Commit message: ガバーデータ生成
Parts:
- R8: value 10kR -> 100kR
- moved TH1 0.10 mm to (143.4, 132.0)
Changed lines of the file:
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@@
 			)
 		)
-		(property "Value" "10kR"
+		(property "Value" "100kR"
 			(at 0 1.43 0)
 			(layer "F.Fab")
@@
 	(footprint "Connector_PinHeader_1.00mm:PinHeader_1x02_P1.00mm_Vertical"
 		(layer "F.Cu")
-		(at 143.5 132 -90)
+		(at 143.4 132 -90)
 		(descr "Through hole straight pin header, 1x02, 1.00mm pitch, single row")
 		(tags "Through hole pin header THT 1x02 1.00mm single row")
@@
 	)
 	(segment
-		(start 149.987 125.563)
-		(end 151 124.55)
+		(start 149.987 127.423668)
+		(end 149.987 125.563)
 		(width 0.2)
 		(layer "B.Cu")
@@
 	)
 	(segment
-		(start 145.410668 132)
-		(end 149.987 127.423668)
+		(start 143.4 132)
+		(end 145.410668 132)
 		(width 0.2)
 		(layer "B.Cu")
@@
 	)
 	(segment
-		(start 143.5 132)
-		(end 145.410668 132)
+		(start 145.410668 132)
+		(end 149.987 127.423668)
 		(width 0.2)
 		(layer "B.Cu")
@@
 	)
 	(segment
-		(start 149.987 127.423668)
-		(end 149.987 125.563)
+		(start 149.987 125.563)
+		(end 151 124.55)
 		(width 0.2)
 		(layer "B.Cu")
@@
 	)
 	(zone
-		(net 14)
-		(net_name "VREF_T1")
-		(layer "F.Cu")
-		(name "$teardrop_padvia$")
-		(hatch full 0.1)
-		(priority 30057)
-		(attr
-			(teardrop
-				(type padvia)
-			)
-		)
-		(connect_pads yes
-			(clearance 0)
-		)
-		(min_thickness 0.0254)
-		(filled_areas_thickness no)
-		(fill yes
-			(thermal_gap 0.5)
-			(thermal_bridge_width 0.5)
-			(island_removal_mode 1)
-			(island_area_min 10)
-		)
-		(polygon
-			(pts
-				(xy 149.620165 121.821586) (xy 149.761586 121.680165) (xy 149.33858 121.091956) (xy 148.866793 121.411293)
-				(xy 149.1175 121.887)
-			)
-		)
-	)
-	(zone
 		(net 3)
 		(net_name "+3.3V")
@@
 	)
 	(zone
-		(net 33)
-		(net_name "Net-(U1-IN+)")
+		(net 14)
+		(net_name "VREF_T1")
 		(layer "F.Cu")
 		(name "$teardrop_padvia$")
 		(hatch full 0.1)
-		(priority 30022)
+		(priority 30002)
 		(attr
 			(teardrop
@@
 		(polygon
 			(pts
-				(xy 128.672951 112.31) (xy 128.672951 112.51) (xy 129.0885 113.16353) (xy 129.5645 112.8765) (xy 129.561815 112.339)
+				(xy 149.620165 121.821586) (xy 149.761586 121.680165) (xy 149.33858 121.091956) (xy 148.866793 121.411293)
+				(xy 149.1175 121.887)
 			)
 		)
 	)
 	(zone
-		(net 3)
-		(net_name "+3.3V")
+		(net 33)
+		(net_name "Net-(U1-IN+)")
 		(layer "F.Cu")
 		(name "$teardrop_padvia$")
 		(hatch full 0.1)
-		(priority 30102)
+		(priority 30022)
 		(attr
 			(teardrop
@@
 		(polygon
 			(pts
-				(xy 122.4605 104.4365) (xy 122.6605 104.4365) (xy 122.8105 104.1865) (xy 122.5605 103.9355) (xy 122.3105 104.1865)
+				(xy 128.672951 112.31) (xy 128.672951 112.51) (xy 129.0885 113.16353) (xy 129.5645 112.8765) (xy 129.561815 112.339)
 			)
 		)
 	)
 	(zone
-		(net 18)
-		(net_name "Net-(J6-Pin_2)")
+		(net 3)
+		(net_name "+3.3V")
 		(layer "F.Cu")
 		(name "$teardrop_padvia$")
 		(hatch full 0.1)
-		(priority 30005)
+		(priority 30102)
 		(attr
 			(teardrop
@@
 		(polygon
 			(pts
-				(xy 141.278 77.897148) (xy 141.678 77.897148) (xy 142.147148 76.42395) (xy 141.338 75.437) (xy 140.652038 76.721345)
+				(xy 122.4605 104.4365) (xy 122.6605 104.4365) (xy 122.8105 104.1865) (xy 122.5605 103.9355) (xy 122.3105 104.1865)
 			)
 		)
 	)
 	(zone
-		(net 5)
-		(net_name "Net-(D4-A)")
+		(net 18)
+		(net_name "Net-(J6-Pin_2)")
 		(layer "F.Cu")
 		(name "$teardrop_padvia$")
 		(hatch full 0.1)
-		(priority 30000)
+		(priority 30005)
 		(attr
 			(teardrop
@@
 		(polygon
 			(pts
-				(xy 175.914 89.038) (xy 175.114 89.038) (xy 174.514 90.059922) (xy 175.514 91.789) (xy 176.514 90.059922)
+				(xy 141.278 77.897148) (xy 141.678 77.897148) (xy 142.147148 76.42395) (xy 141.338 75.437) (xy 140.652038 76.721345)
 			)
 		)
 	)
 	(zone
-		(net 3)
-		(net_name "+3.3V")
+		(net 5)
+		(net_name "Net-(D4-A)")
 		(layer "F.Cu")
 		(name "$teardrop_padvia$")
 		(hatch full 0.1)
-		(priority 30026)
+		(priority 30000)
 		(attr
 			(teardrop
@@
 		(polygon
 			(pts
-				(xy 146.9425 122.362) (xy 147.1425 122.362) (xy 147.511921 121.740387) (xy 147.0425 121.411) (xy 146.573079 121.740387)
+				(xy 175.914 89.038) (xy 175.114 89.038) (xy 174.514 90.059922) (xy 175.514 91.789) (xy 176.514 90.059922)
 			)
 		)
@@
 	)
 	(zone
+		(net 27)
+		(net_name "Net-(U4-IN+)")
+		(layer "F.Cu")
+		(name "$teardrop_padvia$")
+		(hatch full 0.1)
+		(priority 30049)
+		(attr
+			(teardrop
+				(type padvia)
+			)
+		)
+		(connect_pads yes
+			(clearance 0)
+		)
+		(min_thickness 0.0254)
+		(filled_areas_thickness no)
+		(fill yes
+			(thermal_gap 0.5)
+			(thermal_bridge_width 0.5)
+			(island_removal_mode 1)
+			(island_area_min 10)
+		)
+		(polygon
+			(pts
+				(xy 130.4885 104.507) (xy 130.4885 104.307) (xy 129.899604 103.974127) (xy 129.5625 104.407) (xy 129.899604 104.839873)
+			)
+		)
+	)
+	(zone
 		(net 3)
 		(net_name "+3.3V")
@@
 		(name "$teardrop_padvia$")
 		(hatch full 0.1)
-		(priority 30014)
+		(priority 30000)
 		(attr
 			(teardrop
@@
 	)
 	(zone
-		(net 27)
-		(net_name "Net-(U4-IN+)")
+		(net 3)
+		(net_name "+3.3V")
 		(layer "F.Cu")
 		(name "$teardrop_padvia$")
 		(hatch full 0.1)
-		(priority 30049)
+		(priority 30001)
 		(attr
 			(teardrop
@@
 		(polygon
 			(pts
-				(xy 130.4885 104.507) (xy 130.4885 104.307) (xy 129.899604 103.974127) (xy 129.5625 104.407) (xy 129.899604 104.839873)
+				(xy 146.9425 122.362) (xy 147.1425 122.362) (xy 147.511921 121.740387) (xy 147.0425 121.411) (xy 146.573079 121.740387)
 			)
 		)
@@
 	)
 	(zone
-		(net 14)
-		(net_name "VREF_T1")
-		(layer "B.Cu")
-		(name "$teardrop_padvia$")
-		(hatch full 0.1)
-		(priority 30003)
-		(attr
-			(teardrop
-				(type padvia)
-			)
-		)
-		(connect_pads yes
-			(clearance 0)
-		)
-		(min_thickness 0.0254)
-		(filled_areas_thickness no)
-		(fill yes
-			(thermal_gap 0.5)
-			(thermal_bridge_width 0.5)
-			(island_removal_mode 1)
-			(island_area_min 10)
-		)
-		(polygon
-			(pts
-				(xy 144.35 132.1) (xy 144.35 131.9) (xy 143.925 131.575) (xy 143.499 132) (xy 143.925 132.425)
-			)
-		)
-	)
-	(zone
 		(net 3)
 		(net_name "+3.3V")
@@
 			)
 		)
+	)
+	(zone
+		(net 14)
+		(net_name "VREF_T1")
+		(layer "B.Cu")
+		(name "$teardrop_padvia$")
+		(hatch full 0.1)
+		(priority 30000)
+		(attr
+			(teardrop
+				(type padvia)
+			)
+		)
+		(connect_pads yes
+			(clearance 0)
+		)
+		(min_thickness 0.0254)
+		(filled_areas_thickness no)
+		(fill yes
+			(thermal_gap 0.5)
+			(thermal_bridge_width 0.5)
+			(island_removal_mode 1)
+			(island_area_min 10)
+		)
+		(polygon
+			(pts
+				(xy 144.25 132.1) (xy 144.25 131.9) (xy 143.825 131.575) (xy 143.399 132) (xy 143.825 132.425)
+			)
+		)
