File: KiCAD/PowerControlModule/PowerControl.kicad_sch (KiCad schematic)
At the start: 49 parts, among them J1 DF51-2P-2DS, J2 DF51-2P-2DS, Q1 AO3401A, Q2 AO3401A, U2 TPS22810DRV, U3 TPS22810DRV, U4 INA219AxDCN, U5 INA219AxDCN, U6 StarawberryLinux_LTC3118, U7 INA219AxDCN

Commit message: PowerControlModuleを作成．ソフトウェアの開発も進めなければいけない....
Parts:
- removed C1, C2: 1uF, Capacitor_SMD:C_0603_1608Metric_Pad1.08x0.95mm_HandSolder, symbol Device:C
- removed C3, C4: 10uF, Capacitor_SMD:C_0805_2012Metric_Pad1.18x1.45mm_HandSolder, symbol Device:C
- removed C5, C6: 22uF, Capacitor_SMD:C_0805_2012Metric_Pad1.18x1.45mm_HandSolder, symbol Device:C
- removed D1, D2: SB34AFC, Diode_SMD:D_SMA_Handsoldering, symbol Device:D_Schottky
- removed R1, R2: 10kR, Resistor_SMD:R_0603_1608Metric_Pad0.98x0.95mm_HandSolder, symbol Device:R
- removed R3, R4: 120, Resistor_SMD:R_0603_1608Metric_Pad0.98x0.95mm_HandSolder, symbol Device:R
- removed U2, U3: TPS22810DRV, TSRP_IC:DBV0006A_M, symbol TSRP_IC:TPS22810DBVR
- added C1, C3: 2.2uF, Capacitor_SMD:C_0603_1608Metric_Pad1.08x0.95mm_HandSolder, symbol Device:C_Small
- added C2, C4: 22uF, Capacitor_SMD:C_0805_2012Metric_Pad1.18x1.45mm_HandSolder, symbol Device:C_Small
- added Q1, Q3: AO3400A, Package_TO_SOT_SMD:SOT-23_Handsoldering, symbol Simulation_SPICE:NMOS
- added Q2, Q4, Q5, Q6: AO3401A, Package_TO_SOT_SMD:SOT-23_Handsoldering, symbol Transistor_FET:QM6015D
- added R26: 10kR, Resistor_SMD:R_0603_1608Metric_Pad0.98x0.95mm_HandSolder, symbol Device:R
- added R3, R6: 820R, Resistor_SMD:R_0603_1608Metric_Pad0.98x0.95mm_HandSolder, symbol Device:R_Small
- added R4, R7: 10kR, Resistor_SMD:R_0603_1608Metric_Pad0.98x0.95mm_HandSolder, symbol Device:R_Small
- added R5, R8: 100kR, Resistor_SMD:R_0603_1608Metric_Pad0.98x0.95mm_HandSolder, symbol Device:R_Small
- added TH1: Thermistor_NTC, Connector_PinHeader_1.27mm:PinHeader_1x02_P1.27mm_Vertical, symbol Device:Thermistor_NTC
- added U2: MCP1792x-3302xCB, Package_TO_SOT_SMD:SOT-23_Handsoldering, symbol Regulator_Linear:MCP1792x-3302xCB
- Q7: renamed from Q1; footprint Package_TO_SOT_SMD:SOT-23 -> Package_TO_SOT_SMD:SOT-23_Handsoldering
- Q8: renamed from Q2; footprint Package_TO_SOT_SMD:SOT-23 -> Package_TO_SOT_SMD:SOT-23_Handsoldering
- renumbered C12 to C10, C13 to C11, C14 to C12, C7 to C5, C8 to C6, C9 to C7, C10 to C8, C11 to C9, D3 to D1, D4 to D2, D5 to D3, D6 to D4, J2 to J1, J1 to J2, R6 to R10, R7 to R11, R8 to R12, R5 to R13, R10 to R14, R11 to R15, R12 to R16, R13 to R17, R14 to R18, R15 to R19, R16 to R20, R18 to R21, R17 to R22, R19 to R23, U4 to U3, U5 to U4, U6 to U5, U7 to U6
Connections:
- net +3.3V: now also R26.1
- net BATT_IN: now also Q4.3 (S)
- net Battery_ENSW: now also R3.1
- net GND: now also C1.2, C3.2, Q1.3 (S), Q3.3 (S), TH1.2, U2.1 (GND)
- net V1GD: now reaches D1.1 (K), U5.13 (V1GD)
- net at C7.2, U3.2 (IN-): now also R13.2; no longer R13.1
- net VOUT: now reaches C11.1, D4.1 (K), Q7.3 (S), R18.2, R19.1, U5.14 (VOUT), U5.15 (VOUT)
- net BATT: now reaches J2.2 (Pin_2)
- net BATT: now also C2.1, Q2.3 (S), R4.1
- net PGD: now reaches D3.1 (K), U5.11 (PGD)
- net V2GD: now reaches D2.1 (K), U5.12 (V2GD)
- net GPU: now reaches J1.2 (Pin_2)
- net GPU: now also C1.1, C4.1, Q5.3 (S), R7.1, U2.3 (VI)
- net GPU_IN: no longer names the net of R11.1, R9.2
- net GPU_IN: now also Q6.3 (S)
- net GPU_OUT: no longer names the net of R11.2, U5.2 (VIN2), U5.7 (RUN2)
- net GPU_OUT: now also R13.1; no longer R13.2
- new net: C2.2, Q2.1 (G), Q4.1 (G), R4.2, R5.1
- new net: Q2.2 (D), Q4.2 (D)
- new net: C4.2, Q5.1 (G), Q6.1 (G), R7.2, R8.1
- new net: Q1.1 (D), R5.2
- new net: Q1.2 (G), R3.2
- new net: C3.1, R6.1, U2.2 (VO)
- new net: Q5.2 (D), Q6.2 (D)
- new net: Q3.1 (D), R8.2
- new net: Q3.2 (G), R6.2
- new net VREF_T1: R26.2, TH1.1
Other:
- note added: "逆流防止ロードスイッチ"
- note removed: "CTピン：VOUTの立ち上がり時間を制御できる 3.215 ~ 2.085 ms の間 今回の使い方だとあまり意味ない"
- note removed: "逆接続保護ダイオード"
- moved on the sheet: J1, J2, R13

Commit message: PowerModule，Build-2完成．発注．
Parts:
- TH1: footprint Connector_PinHeader_1.27mm:PinHeader_1x02_P1.27mm_Vertical -> (none)
Changed lines of the file:
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@@
 			)
 		)
-		(property "Footprint" "Connector_PinHeader_1.27mm:PinHeader_1x02_P1.27mm_Vertical"
+		(property "Footprint" ""
 			(at 167.64 140.97 0)
 			(effects
@@
 			)
 		)
-		(property "Datasheet" "~"
+		(property "Datasheet" "https://akizukidenshi.com/catalog/g/g105251/"
 			(at 167.64 140.97 0)
 			(effects
@@
 			)
 		)
-		(property "Datasheet" ""
+		(property "Datasheet" "https://strawberry-linux.com/catalog/items?code=13118"
 			(at 161.29 59.69 0)
 			(effects
