File: KiCAD/PowerControlModule/PowerControl.kicad_sch (KiCad schematic)
At the start: 54 parts, among them J1 DF51-2P-2DS, J2 DF51-2P-2DS, Q11 Si4162DY, Q12 Si4162DY, Q2 AO3401A, Q3 AO3400A, Q4 AO3401A, Q5 AO3401A, Q6 AO3401A, Q7 AO3401A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

Commit message: Build-3発注した
Parts:
- added C1: 100uF, Capacitor_THT:CP_Radial_D6.3mm_P2.50mm, symbol Device:C_Polarized
- added R22: 10kR, Resistor_SMD:R_0603_1608Metric_Pad0.98x0.95mm_HandSolder, symbol Device:R_Small
- R4: value 10kR -> 5.6kR
- R5: value 100kR -> 3.3kR
- R8: value 100kR -> 4.7kR
Connections:
- net BUS_LOWER: now also C1.1
- net GND: now also C1.2, R22.2
- net at Q3.1 (G), R17.2: now also R22.1
Other:
- note added: "15Vくらい"
- note added: "17V"
- note added: "R4, R5 で分圧して5.5Vくらい"
- note added: "R7, R8 で分圧して5.5Vくらい"
- moved on the sheet: R17

Commit message: MOSFETのフットプリントを修正
Parts:
- removed Q2, Q4, Q5, Q6, Q7, Q8: AO3401A, Package_TO_SOT_SMD:SOT-23_Handsoldering, symbol Transistor_FET:QM6015D
- added Q1, Q2, Q4, Q5, Q7, Q9: AO3401A, Package_TO_SOT_SMD:SOT-23_Handsoldering, symbol Transistor_FET:AO3401A
- added Q10, Q6: AO3401A, Package_TO_SOT_SMD:SOT-23, symbol Transistor_FET:AO3401A
- TH1: footprint Connector_PinHeader_1.27mm:PinHeader_1x02_P1.27mm_Vertical -> Connector_PinHeader_2.00mm:PinHeader_1x02_P2.00mm_Vertical
Connections:
- net +VSW: now also Q7.2 (S)
- net BATT: now also Q2.2 (S)
- net BATT_UPPER: now also Q4.2 (S)
- net GPU: now also Q5.2 (S)
- net GPU_UPPER: now also Q9.2 (S)
- net at C11.1, D4.1 (K), Q11.5 (D)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: now also Q1.2 (S)
- net at C2.2, R4.2, R5.1: now also Q2.1 (G), Q4.1 (G)
- net at C4.2, R7.2, R8.1: now also Q5.1 (G), Q9.1 (G)
- net at C11.2, R19.2, R20.1: now also Q1.1 (G), Q7.1 (G)
- new net: Q1.3 (D), Q7.3 (D)
- new net: Q2.3 (D), Q4.3 (D)
- new net: Q5.3 (D), Q9.3 (D)
Other:
- note added: "1:G"
- note added: "2:S"
- note added: "3:D"
- note added: "AO3401A"
- note added: "今までの接続 H-59 H-60"

Commit message: Build-4作成完了
Parts:
- J1, J2: value DF51-2P-2DS -> DF1B-2S-2.5R; footprint TSRP_Connector_Hirose:DF51-2P-2DS -> TSRP_Connector:DF1B-2S-2.5R
- Q10, Q6: now not fitted
Other:
- note added: "Pch MOSFET"
Changed lines of the file:
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@@
 		)
 	)
+	(text "Pch MOSFET"
+		(exclude_from_sim no)
+		(at 103.124 2.286 0)
+		(effects
+			(font
+				(size 1.27 1.27)
+			)
+		)
+	)
 	(text "From\nBattery Module\n(Internal)"
 		(exclude_from_sim no)
@@
 		(in_bom no)
 		(on_board no)
-		(dnp no)
+		(dnp yes)
 		(property "Reference" "Q10"
 			(at 68.58 -19.05 90)
@@
 	)
 	(symbol
+		(lib_name "AO3401A_1")
 		(lib_id "Transistor_FET:AO3401A")
 		(at 55.88 43.18 270)
@@
 			)
 		)
-		(property "Value" "DF51-2P-2DS"
+		(property "Value" "DF1B-2S-2.5R"
 			(at 27.94 119.3799 90)
 			(effects
@@
 			)
 		)
-		(property "Footprint" "TSRP_Connector_Hirose:DF51-2P-2DS"
+		(property "Footprint" "TSRP_Connector:DF1B-2S-2.5R"
 			(at 22.86 118.11 0)
 			(effects
@@
 			)
 		)
-		(property "Value" "DF51-2P-2DS"
+		(property "Value" "DF1B-2S-2.5R"
 			(at 27.686 34.29 90)
 			(effects
@@
 			)
 		)
-		(property "Footprint" "TSRP_Connector_Hirose:DF51-2P-2DS"
+		(property "Footprint" "TSRP_Connector:DF1B-2S-2.5R"
 			(at 22.86 33.02 0)
 			(effects
@@
 	)
 	(symbol
+		(lib_name "AO3401A_2")
 		(lib_id "Transistor_FET:AO3401A")
 		(at 67.31 43.18 90)
@@
 		(in_bom no)
 		(on_board no)
-		(dnp no)
+		(dnp yes)
 		(property "Reference" "Q6"
 			(at 82.55 -19.05 90)

Commit message: Build-5を作成
Parts:
- C1: value 100uF -> 220uF
- C21: value 0.0056uF -> 0.056uF
- D3: value Orange -> Green
Changed lines of the file:
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@@
 	)
 	(symbol
+		(lib_name "AO3401A_5")
 		(lib_id "Transistor_FET:AO3401A")
 		(at 267.97 43.18 90)
@@
 	)
 	(symbol
+		(lib_name "AO3401A_3")
 		(lib_id "Transistor_FET:AO3401A")
 		(at 67.31 129.54 270)
@@
 			)
 		)
-		(property "Value" "Orange"
+		(property "Value" "Green"
 			(at 167.64 120.5864 90)
 			(effects
@@
 			)
 		)
-		(property "Value" "100uF"
+		(property "Value" "220uF"
 			(at 219.71 112.1409 0)
 			(effects
@@
 	)
 	(symbol
+		(lib_name "AO3401A_4")
 		(lib_id "Transistor_FET:AO3401A")
 		(at 78.74 129.54 90)
@@
 	)
 	(symbol
+		(lib_name "AO3401A_6")
 		(lib_id "Transistor_FET:AO3401A")
 		(at 256.54 43.18 270)
@@
 			)
 		)
-		(property "Value" "0.0056uF"
+		(property "Value" "0.056uF"
 			(at 158.7563 90.17 90)
 			(effects

Commit message: 修正した．発注する．
Parts:
- removed D3: Green, LED_SMD:LED_0603_1608Metric_Pad1.05x0.95mm_HandSolder, symbol Device:LED_Small
- removed R21: 3.6kR, Resistor_SMD:R_0603_1608Metric_Pad0.98x0.95mm_HandSolder, symbol Device:R_Small
- added R27: 10k, Resistor_SMD:R_0603_1608Metric, symbol Device:R_Small
Connections:
- net +3.3V: now also R27.1
- net LTC3119_PGOOD: now reaches U11.2 (PGOOD)
- net LTC3119_PGOOD: now also R27.2
