File: KiCAD/PowerControlModule/PowerControlModule.kicad_pcb (KiCad board)
At the start: 2 copper layers, 90 x 70 mm, 71 parts, among them J1 DF51-2P-2DS, J2 DF51-2P-2DS, J3 DF11-8DP-2DS, Q1 AO3401A, Q2 AO3401A, U1 XIAO-RP2040-DIP, U2 TPS22810DRV, U3 TPS22810DRV, U4 INA219AxDCN, U5 INA219AxDCN, U6 StarawberryLinux_LTC3118, U7 INA219AxDCN, U8 MCP2515-xSO, U9 MCP2562-E-SN, Y1 8MHz

Commit message: PowerControlModuleを作成．ソフトウェアの開発も進めなければいけない....
Parts:
- removed the C5 at (148.1, 86.6)
- removed the C6 at (143.8, 116.1)
- removed the D1 at (145.4, 73.0)
- removed the D2 at (129.3, 127.0)
- removed the R1 at (139.1, 80.8)
- removed the R2 at (132.1, 117.3)
- removed the U3 at (137.4, 116.1)
- added C19: 2.2uF, Capacitor_SMD:C_0603_1608Metric_Pad1.08x0.95mm_HandSolder, F.Cu at (161.2, 117.1)
- added Q1: AO3400A, Package_TO_SOT_SMD:SOT-23_Handsoldering, F.Cu at (129.0, 123.6)
- added Q2: AO3401A, Package_TO_SOT_SMD:SOT-23_Handsoldering, F.Cu at (137.3, 119.1)
- added Q3: AO3400A, Package_TO_SOT_SMD:SOT-23_Handsoldering, F.Cu at (134.4, 85.6)
- added Q4: AO3401A, Package_TO_SOT_SMD:SOT-23_Handsoldering, F.Cu at (133.4, 116.1)
- added Q5: AO3401A, Package_TO_SOT_SMD:SOT-23_Handsoldering, F.Cu at (144.3, 80.5)
- added Q6: AO3401A, Package_TO_SOT_SMD:SOT-23_Handsoldering, F.Cu at (148.6, 83.5)
- added R26: 10kR, Resistor_SMD:R_0603_1608Metric_Pad0.98x0.95mm_HandSolder, F.Cu at (147.6, 124.5)
- added R5: 100kR, Resistor_SMD:R_0603_1608Metric_Pad0.98x0.95mm_HandSolder, F.Cu at (130.0, 118.6)
- added R6: 820R, Resistor_SMD:R_0603_1608Metric_Pad0.98x0.95mm_HandSolder, F.Cu at (134.4, 82.9)
- added R7: 10kR, Resistor_SMD:R_0603_1608Metric_Pad0.98x0.95mm_HandSolder, F.Cu at (140.8, 79.5)
- added R8: 100kR, Resistor_SMD:R_0603_1608Metric_Pad0.98x0.95mm_HandSolder, F.Cu at (140.8, 83.6)
- added TH1: Thermistor_NTC, Connector_PinHeader_1.27mm:PinHeader_1x02_P1.27mm_Vertical, F.Cu at (149.7, 124.5)
- added U9: MCP1792x-5002xCB, Package_TO_SOT_SMD:SOT-23_Handsoldering, F.Cu at (162.2, 114.4)
- C1: value 1uF -> 2.2uF
- C2: value 1uF -> 22uF; footprint Capacitor_SMD:C_0603_1608Metric_Pad1.08x0.95mm_HandSolder -> Capacitor_SMD:C_0805_2012Metric_Pad1.18x1.45mm_HandSolder
- C20: value 330uF -> 2.2uF; footprint Capacitor_SMD:CP_Elec_10x10 -> Capacitor_SMD:C_0603_1608Metric_Pad1.08x0.95mm_HandSolder
- C3: value 10uF -> 2.2uF; footprint Capacitor_SMD:C_0805_2012Metric_Pad1.18x1.45mm_HandSolder -> Capacitor_SMD:C_0603_1608Metric_Pad1.08x0.95mm_HandSolder
- C4: value 10uF -> 22uF
- Q7: renamed from Q1; footprint Package_TO_SOT_SMD:SOT-23 -> Package_TO_SOT_SMD:SOT-23_Handsoldering
- Q8: renamed from Q2; footprint Package_TO_SOT_SMD:SOT-23 -> Package_TO_SOT_SMD:SOT-23_Handsoldering
- R3: value 120 -> 820R
- R4: value 120 -> 10kR
- U2: value TPS22810DRV -> MCP1792x-3302xCB; footprint TSRP_IC:DBV0006A_M -> Package_TO_SOT_SMD:SOT-23_Handsoldering
- moved C20 44.5 mm to (163.2, 111.4), turned to 180 degrees
- moved C4 40.6 mm to (138.4, 79.8), turned to -90 degrees
- moved R3 35.3 mm to (128.0, 118.5), turned to -90 degrees
- moved R19 29.3 mm to (184.9, 96.4), turned to -90 degrees
- moved R16 21.1 mm to (149.7, 71.8), turned to 90 degrees
- moved R18 14.3 mm to (178.6, 91.7)
- moved R1 11.5 mm to (129.8, 112.5), turned to 180 degrees
- moved D6 10.9 mm to (127.5, 83.6), turned to 90 degrees
- moved C2 10.6 mm to (142.2, 120.2), turned to 90 degrees
- moved U2 10.6 mm to (133.7, 78.5), turned to 0 degrees
- moved U6 10.4 mm to (144.4, 115.8), turned to 180 degrees
- moved C10 10.2 mm to (146.4, 113.3), turned to 180 degrees
- moved C11 9.97 mm to (187.8, 88.0), turned to 90 degrees
- moved C1 9.76 mm to (134.4, 75.6)
- moved R2 9.07 mm to (129.8, 110.1), turned to 180 degrees
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- renumbered C12 to C10, C13 to C11, C14 to C12, C15 to C13, C16 to C14, C17 to C15, C18 to C16, C19 to C17, C7 to C5, C8 to C6, C9 to C7, C10 to C8, C11 to C9, D3 to D1, D4 to D2, D5 to D3, D6 to D4, D7 to D5, D8 to D6, J2 to J1, J1 to J2, R22 to R1, R6 to R10, R7 to R11, R8 to R12, R5 to R13, R10 to R14, R11 to R15, R12 to R16, R13 to R17, R14 to R18, R15 to R19, R23 to R2, R16 to R20, R18 to R21, R17 to R22, R19 to R23, R20 to R24, R21 to R25, U4 to U3, U5 to U4, U6 to U5, U7 to U6, U8 to U7, U9 to U8
Connections:
- net Net-(D3-K) renamed V1GD
- net Net-(D4-K) renamed V2GD
- net Net-(D5-K) renamed PGD
- C1 pad 1: Net-(D1-K) -> /PowerControl/GPU
- C11 pad 1: Net-(D6-K) (its old number) -> /PowerControl/VOUT
- C17 pad 2: +5V -> +5VD
- C2 pad 1: Net-(D2-K) -> /PowerControl/BATT
- C2 pad 2: GND -> Net-(Q2-G)
- C20 pad 1: +12V -> +5VD
- C3 pad 1: Net-(U2-CT) -> Net-(U2-VO)
- C4 pad 1: Net-(U3-CT) -> /PowerControl/GPU
- C4 pad 2: GND -> Net-(Q5-G)
- C7 pad 2: Net-(U4-IN-) (its old number) -> Net-(U3-IN-)
- D4 pad 1: Net-(D6-K) (its old number) -> /PowerControl/VOUT
- J1 pad 2: Net-(D1-A) (its old number) -> /PowerControl/GPU
- J2 pad 2: Net-(D2-A) (its old number) -> /PowerControl/BATT
- Q7 pad 3: Net-(D6-K) (its old number) -> /PowerControl/VOUT
- R11 pad 1: /PowerControl/GPU_IN -> Net-(Q6-S)
- R11 pad 2: /PowerControl/GPU_OUT -> Net-(U5-RUN2)
- R13 pad 1: Net-(U4-IN-) (its old number) -> Net-(U5-RUN2)
- R13 pad 2: /PowerControl/GPU_OUT -> Net-(U3-IN-)
- R18 pad 2: Net-(D6-K) (its old number) -> /PowerControl/VOUT
- R19 pad 1: Net-(D6-K) (its old number) -> /PowerControl/VOUT
- R3 pad 1: Net-(U2-QOD) -> Battery_ENSW
- R3 pad 2: /PowerControl/GPU_IN -> Net-(Q1-G)
- R4 pad 1: Net-(U3-QOD) -> /PowerControl/BATT
- R4 pad 2: /PowerControl/BATT_IN -> Net-(Q2-G)
- R9 pad 2: /PowerControl/GPU_IN -> Net-(Q6-S)
- U1 pad 3: GPU_ENSW -> VREF_T1
- U2 pad 1: Net-(D1-K) -> GND
- U2 pad 2: GND -> Net-(U2-VO)
- U2 pad 3: GPU_ENSW -> /PowerControl/GPU
- U3 pad 2: Net-(U4-IN-) (its old number) -> Net-(U3-IN-)
- U5 pad 14: Net-(D6-K) (its old number) -> /PowerControl/VOUT
- U5 pad 15: Net-(D6-K) (its old number) -> /PowerControl/VOUT
- U5 pad 2: /PowerControl/GPU_OUT -> Net-(U5-RUN2)
- U5 pad 7: /PowerControl/GPU_OUT -> Net-(U5-RUN2)
- U8 pad 3: +5V -> +5VD
Routing:
- net +12V: track 24.1 -> 194.0 mm, vias 2 -> 0
- net +3.3V: track 0.00 -> 128.4 mm, vias 0 -> 5
- net SPI_CS_MCP2515: track 0.00 -> 73.5 mm, vias 0 -> 2
- net SPI_MOSI: track 0.00 -> 71.6 mm, vias 0 -> 2
- net SPI_MISO: track 0.00 -> 68.8 mm, vias 0 -> 2
- net V1GD: track 0.00 -> 68.1 mm, vias 0 -> 1
- net SPI_SCK: track 0.00 -> 65.4 mm, vias 0 -> 2
- net I2C_SDA: track 0.00 -> 55.0 mm, vias 0 -> 4
- net V2GD: track 0.00 -> 51.0 mm, vias 0 -> 1
- net I2C_SCL: track 0.00 -> 49.7 mm, vias 0 -> 4
- net VREF_T1: track 0.00 -> 43.3 mm, vias 0 -> 2
- net /PowerControl/BUS_IN: track 8.52 -> 41.1 mm, vias 0 -> 2
- net Net-(Q7-G): track 0.00 -> 30.2 mm, vias 0 -> 3
- net PGD: track 2.50 -> 31.0 mm
- net Net-(U5-RUN2): track 0.00 -> 28.0 mm
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- added copper zone on F.Cu, net +12V
- added copper zone on F.Cu, net /PowerControl/BATT
- added copper zone on F.Cu, net /PowerControl/BATT_OUT
- added copper zone on F.Cu, net /PowerControl/BUS_IN
- added copper zone on F.Cu, net /PowerControl/VOUT
- added copper zone on F.Cu, net Net-(Q6-S)
- added copper zone on F.Cu, net Net-(U5-RUN2)
Other:
- board text added: "0b100 0000"
- board text added: "0b100 0001"
- board text added: "0b100 0101"
- board text added: "BATT"
- board text added: "BUS"
- board text added: "EXT"
- board text added: "M78AR05-0.5"

Commit message: PowerModule，Build-2完成．発注．
Parts:
- added G***: LOGO, LOGO, B.Cu at (135.6, 131.6)
- added G***: LOGO, LOGO, B.Cu at (165.2, 131.6)
- moved J2 0.54 mm to (137.0, 134.2)
- moved C2 0.30 mm to (142.2, 119.9)
Routing:
- net GND: vias 143 -> 165
Other:
- board text added: "17V IN"
- board text added: "Power Module Build-2"
- board text added: "SUBARU"
- board text added: "Tokai Student Rocket Project"
- board text added: "V1.3"

Commit message: Build-3完成．本日発注．
Parts:
- removed C1: 2.2uF, Capacitor_SMD:C_0603_1608Metric_Pad1.08x0.95mm_HandSolder
- removed C12, C6, C7, C8: 0.1uF, Capacitor_SMD:C_0603_1608Metric_Pad1.08x0.95mm_HandSolder
- removed Q1: AO3400A, Package_TO_SOT_SMD:SOT-23_Handsoldering
- removed R22: 10R, Resistor_SMD:R_0603_1608Metric_Pad0.98x0.95mm_HandSolder
- removed R23: 0.1R, Resistor_SMD:R_2816_7142Metric_Pad3.20x4.45mm_HandSolder
- removed U2: MCP1792x-3302xCB, Package_TO_SOT_SMD:SOT-23_Handsoldering
- added C18: 0.056uF, Inductor_SMD:L_0603_1608Metric, F.Cu at (153.2, 98.0)
- added C21: 0.0056uF, Inductor_SMD:L_0603_1608Metric, F.Cu at (153.2, 101.6)
- added C22: 0.1uF, Capacitor_SMD:C_0603_1608Metric_Pad1.08x0.95mm_HandSolder, F.Cu at (152.4, 120.7)
- added D7: Red, LED_SMD:LED_0603_1608Metric_Pad1.05x0.95mm_HandSolder, F.Cu at (152.4, 115.1)
- added D8: Red, LED_SMD:LED_0603_1608Metric_Pad1.05x0.95mm_HandSolder, F.Cu at (145.5, 100.6)
- added D9: Red, LED_SMD:LED_0603_1608Metric_Pad1.05x0.95mm_HandSolder, F.Cu at (133.9, 99.8)
- added Q11: Si4162DY, Package_SO:SOIC-8_3.9x4.9mm_P1.27mm, F.Cu at (153.9, 91.9)
- added Q12: Si4162DY, Package_SO:SOIC-8_3.9x4.9mm_P1.27mm, F.Cu at (153.2, 107.4)
- added U11: LTC3119, TSRP_IC:StrawberryLinux_LTC3119, F.Cu at (174.2, 93.0)
- C10: footprint Capacitor_SMD:C_0603_1608Metric_Pad1.08x0.95mm_HandSolder -> Capacitor_SMD:C_0603_1608Metric
- C3: value 2.2uF -> 0.1uF
- D4: value SR54F -> SMAJ45A; footprint Diode_SMD:D_SMB_Handsoldering -> Diode_SMD:D_SMA
- D5: value GS1010FL -> SMAJ45A; footprint Diode_SMD:D_SOD-123 -> Diode_SMD:D_SMA
- Q3: footprint Package_TO_SOT_SMD:SOT-23_Handsoldering -> Package_TO_SOT_SMD:TSOT-23_HandSoldering
- R10: value 10R -> 15mR; footprint Resistor_SMD:R_0603_1608Metric_Pad0.98x0.95mm_HandSolder -> Resistor_SMD:R_2512_6332Metric_Pad1.40x3.35mm_HandSolder
- R11, R12: value 0.1R -> 15mR; footprint Resistor_SMD:R_2816_7142Metric_Pad3.20x4.45mm_HandSolder -> Resistor_SMD:R_2512_6332Metric_Pad1.40x3.35mm_HandSolder
- R13, R14, R9: value 10R -> 680R
- R15, R16: value 2.4kR -> 2.7kR
- R17: value 2.4kR -> 820
- R21: value 10R -> 3.6kR
- R24: value 10K -> 10kR
- R25: value 120 -> 120R
- R3, R6: value 820R -> 10kR
- U3, U4, U6: value INA219AxDCN -> INA228; footprint Package_TO_SOT_SMD:SOT-23-8 -> Package_SO:VSSOP-10_3x3mm_P0.5mm
- U5: value StarawberryLinux_LTC3118 -> LTC4353; footprint TSRP_IC:StrawberryLinux_LTC3118 -> Package_SO:MSOP-16_3x4.039mm_P0.5mm
- Y1: footprint Crystal:Crystal_SMD_HC49-SD -> Crystal:Crystal_HC49-4H_Vertical
- moved D1 64.6 mm to (168.9, 68.6), turned to 0 degrees
- moved R15 54.4 mm to (168.9, 75.7), turned to 0 degrees
- moved R17 36.3 mm to (134.1, 117.0), turned to 0 degrees
- moved Q3 34.2 mm to (134.9, 119.8), turned to 0 degrees
- moved D4 31.4 mm to (150.6, 85.3), turned to 180 degrees
- moved R20 29.4 mm to (166.1, 86.4), turned to -90 degrees
- moved C11 28.7 mm to (159.3, 85.3), turned to 0 degrees
- moved R18 28.2 mm to (150.6, 87.9), turned to 0 degrees
- moved R6 27.9 mm to (135.1, 110.7), turned to 180 degrees
- moved R9 23.2 mm to (152.4, 113.5), turned to 180 degrees
- moved Q7 21.7 mm to (168.1, 89.9), turned to 180 degrees
- moved C3 21.7 mm to (140.0, 102.1), turned to 90 degrees
- moved Q8 21.1 mm to (171.2, 86.4), turned to 0 degrees
- moved R21 20.1 mm to (169.4, 125.0), turned to -90 degrees
- moved C10 19.1 mm to (147.1, 94.2)
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Connections:
- C10 pad 1: GND -> Net-(U5-VCC)
- C10 pad 2: +3.3V -> GND
- C11 pad 1: /PowerControl/VOUT -> Net-(D4-K)
- C3 pad 1: Net-(U2-VO) -> +3.3V
- D1 pad 1: V1GD -> Net-(D1-K)
- D2 pad 1: V2GD -> Net-(D2-K)
- D3 pad 1: PGD -> Net-(D3-K)
- D4 pad 1: /PowerControl/VOUT -> Net-(D4-K)
- Q3 pad 1: Net-(Q3-D) -> Net-(Q3-G)
- Q3 pad 2: Net-(Q3-G) -> GND
- Q3 pad 3: GND -> Net-(Q3-D)
- Q4 pad 3: /PowerControl/BATT_IN -> /PowerControl/BATT_UPPER
- Q6 pad 3: Net-(Q6-S) -> /PowerControl/GPU_UPPER
- Q7 pad 3: /PowerControl/VOUT -> Net-(D4-K)
- Q8 pad 3: /PowerControl/BUS_IN -> +VSW
- R10 pad 1: Net-(U4-IN+) -> /PowerControl/GPU_UPPER
- R10 pad 2: /PowerControl/BATT_IN -> /PowerControl/GPU_LOWER
- R11 pad 1: Net-(Q6-S) -> /PowerControl/BATT_LOWER
- R11 pad 2: Net-(U5-RUN2) -> /PowerControl/BATT_UPPER
- R12 pad 1: /PowerControl/BATT_IN -> /PowerControl/BUS_LOWER
- R12 pad 2: /PowerControl/BATT_OUT -> +12V
- R13 pad 1: Net-(U5-RUN2) -> Net-(D8-K)
- R13 pad 2: Net-(U3-IN-) -> Net-(U4-~{Alert})
- R14 pad 1: /PowerControl/BATT_OUT -> Net-(D9-K)
- R14 pad 2: Net-(U4-IN-) -> Net-(U3-~{Alert})
- R15 pad 1: +12V -> Net-(D1-A)
- R15 pad 2: Net-(D1-A) -> Net-(D4-K)
- R16 pad 1: +12V -> Net-(D2-A)
- R16 pad 2: Net-(D2-A) -> Net-(D4-K)
- R17 pad 1: +12V -> BATT_EN
- R17 pad 2: Net-(D3-A) -> Net-(Q3-G)
- R18 pad 2: /PowerControl/VOUT -> Net-(D4-K)
- R19 pad 1: /PowerControl/VOUT -> Net-(D4-K)
- R21 pad 1: Net-(U6-IN+) -> +12V
- R21 pad 2: /PowerControl/BUS_IN -> Net-(D3-A)
- R3 pad 1: Battery_ENSW -> LTC4353_EN1
- R3 pad 2: Net-(Q1-G) -> GND
- R5 pad 2: Net-(Q1-D) -> Net-(Q3-D)
- R6 pad 1: Net-(U2-VO) -> LTC4353_EN2
- R6 pad 2: Net-(Q3-G) -> GND
- R8 pad 2: Net-(Q3-D) -> GND
- R9 pad 1: Net-(U3-IN+) -> Net-(D7-K)
- R9 pad 2: Net-(Q6-S) -> Net-(U6-~{Alert})
- U1 pad 2: Battery_ENSW -> VREF_T1
- U1 pad 3: VREF_T1 -> LTC4353_EN1
- U1 pad 4: unconnected-(U1-GPIO29/ADC3/A3-Pad4) -> LTC4353_EN2
- U1 pad 7: unconnected-(U1-GPIO0/TX-Pad7) -> BATT_EN
- U3 pad 1: Net-(U3-IN+) -> GND
- U3 pad 2: Net-(U3-IN-) -> GND
- U3 pad 3: GND -> Net-(U3-~{Alert})
- U3 pad 4: +3.3V -> I2C_SDA
- U3 pad 6: I2C_SDA -> +3.3V
- U3 pad 8: GND -> /PowerControl/GPU_UPPER
- U4 pad 1: Net-(U4-IN+) -> GND
- U4 pad 2: Net-(U4-IN-) -> +3.3V
- U4 pad 3: GND -> Net-(U4-~{Alert})
- U4 pad 4: +3.3V -> I2C_SDA
- U4 pad 6: I2C_SDA -> +3.3V
- U4 pad 7: +3.3V -> GND
- U4 pad 8: GND -> /PowerControl/BATT_UPPER
- U5 pad 1: GND -> LTC4353_EN2
- U5 pad 10: Net-(U5-MODE) -> Net-(D4-K)
- U5 pad 11: PGD -> Net-(U5-CPO1)
- U5 pad 12: V2GD -> Net-(Q11-G)
- U5 pad 13: V1GD -> /PowerControl/GPU_LOWER
- U5 pad 14: /PowerControl/VOUT -> Net-(U5-VCC)
- U5 pad 15: /PowerControl/VOUT -> GND
- U5 pad 16: GND -> LTC4353_EN1
- U5 pad 2: Net-(U5-RUN2) -> (no net)
- U5 pad 3: /PowerControl/BATT_OUT -> (no net)
- U5 pad 4: GND -> /PowerControl/BATT_LOWER
- U5 pad 5: GND -> Net-(Q12-G)
- U5 pad 6: /PowerControl/BATT_OUT -> Net-(U5-CPO2)
- U5 pad 7: Net-(U5-RUN2) -> Net-(D4-K)
- U5 pad 8: Net-(U5-MODE) -> Net-(D2-K)
- U5 pad 9: Net-(U5-MODE) -> Net-(D1-K)
- U6 pad 1: Net-(U6-IN+) -> +3.3V
- U6 pad 2: Net-(U6-IN-) -> +3.3V
- U6 pad 3: GND -> Net-(U6-~{Alert})
- U6 pad 4: +3.3V -> I2C_SDA
- U6 pad 6: I2C_SDA -> +3.3V
- U6 pad 7: +3.3V -> GND
- U6 pad 8: +3.3V -> /PowerControl/BUS_LOWER
Routing:
- net +12V: track 194.0 -> 117.8 mm, vias 0 -> 2
- net V1GD: track 68.1 -> 0.00 mm, vias 1 -> 0
- net LTC4353_EN1: track 0.00 -> 53.1 mm, vias 0 -> 5
- net V2GD: track 51.0 -> 0.00 mm, vias 1 -> 0
- net BATT_EN: track 0.00 -> 50.4 mm, vias 0 -> 2
- net LTC4353_EN2: track 0.00 -> 47.1 mm, vias 0 -> 5
- net Net-(D4-K): track 0.00 -> 44.3 mm
- net /PowerControl/BUS_IN: track 41.1 -> 0.00 mm, vias 2 -> 0
- net Net-(D2-K): track 0.00 -> 41.0 mm, vias 0 -> 2
- net Net-(D3-K): track 0.00 -> 37.3 mm, vias 0 -> 1
- net Net-(D1-K): track 0.00 -> 37.0 mm, vias 0 -> 2
- net Net-(U11-MPPC): track 0.00 -> 33.7 mm
- net PGD: track 31.0 -> 0.00 mm, vias 1 -> 0
- net Net-(U5-RUN2): track 28.0 -> 0.00 mm
- net Battery_ENSW: track 20.9 -> 0.00 mm
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- added copper zone on F.Cu, net +VSW
- added copper zone on F.Cu, net /PowerControl/BATT_LOWER
- added copper zone on F.Cu, net /PowerControl/BATT_UPPER
- added copper zone on F.Cu, net /PowerControl/BUS_LOWER
- added copper zone on F.Cu, net /PowerControl/GPU
- added copper zone on F.Cu, net /PowerControl/GPU_LOWER
- added copper zone on F.Cu, net /PowerControl/GPU_UPPER
- added copper zone on F.Cu, net Net-(D4-K)
- added copper zone on F.Cu, net Net-(Q2-D)
- added copper zone on F.Cu, net Net-(Q5-D)
- added copper zone on F.Cu, net Net-(Q7-D)
- removed copper zone on F.Cu, net /PowerControl/BATT_IN
- removed copper zone on F.Cu, net /PowerControl/BATT_OUT
- removed copper zone on F.Cu, net /PowerControl/BUS_IN
- removed copper zone on F.Cu, net /PowerControl/VOUT
- removed copper zone on F.Cu, net Net-(Q6-S)
- removed copper zone on F.Cu, net Net-(U5-RUN2)
Other:
- board text added: "Power Module Build-3"
- board text added: "SOURCE"
- board text removed: "Power Module Build-2"

Commit message: Build-3発注した
Parts:
- added C1: 100uF, Capacitor_THT:CP_Radial_D6.3mm_P2.50mm, F.Cu at (173.4, 108.5)
- added R22: 10kR, Resistor_SMD:R_0603_1608Metric_Pad0.98x0.95mm_HandSolder, F.Cu at (134.1, 114.2)
- R4: value 10kR -> 5.6kR
- R5: value 100kR -> 3.3kR
- R8: value 100kR -> 4.7kR
- moved C14 1.40 mm to (185.3, 107.8)
- moved U11 1.09 mm to (174.2, 91.9)
- moved C15 0.90 mm to (185.3, 121.8)
Connections:
- H1 pad 1: (no net) -> GND
- H2 pad 1: (no net) -> GND
- H3 pad 1: (no net) -> GND
- H4 pad 1: (no net) -> GND
Routing:
- net Net-(D3-K): track 37.3 -> 42.7 mm
- net Net-(Q3-G): track 2.61 -> 5.40 mm
- net OSC1: track 12.9 -> 11.6 mm
- net OSC2: track 12.4 -> 11.6 mm
- net GND: vias 224 -> 225
Other:
- board text added: "NTC"

Commit message: MOSFETのフットプリントを修正
Parts:
- removed Q6, Q8: AO3401A, Package_TO_SOT_SMD:SOT-23_Handsoldering
- added Q1: AO3401A, Package_TO_SOT_SMD:SOT-23, F.Cu at (1.96, 1.90)
- added Q1: AO3401A, Package_TO_SOT_SMD:SOT-23_Handsoldering, F.Cu at (168.2, 89.9)
- added Q9: AO3401A, Package_TO_SOT_SMD:SOT-23_Handsoldering, F.Cu at (135.0, 86.7)
- TH1: footprint Connector_PinHeader_1.27mm:PinHeader_1x02_P1.27mm_Vertical -> Connector_PinHeader_2.00mm:PinHeader_1x02_P2.00mm_Vertical
- moved R8 7.50 mm to (133.1, 82.7), turned to -90 degrees
- moved R7 6.55 mm to (142.3, 82.9), turned to -90 degrees
- moved R19 5.28 mm to (173.6, 89.9), turned to 180 degrees
- moved Q5 5.15 mm to (138.0, 82.9), turned to 180 degrees
- moved Q7 4.68 mm to (171.2, 86.4)
- moved C4 3.34 mm to (134.1, 79.7), turned to 180 degrees
- moved C2 1.84 mm to (140.8, 119.0), turned to 90 degrees
- moved R20 1.83 mm to (166.1, 84.5), turned to 90 degrees
- moved R5 1.05 mm to (136.9, 116.1)
- moved R4 0.98 mm to (139.0, 118.8), turned to 90 degrees
- moved R6 0.56 mm to (135.1, 110.2)
- moved Q2 0.10 mm to (143.9, 116.6), turned to 90 degrees
- moved Q4 0.05 mm to (139.7, 113.6), turned to -90 degrees
Connections:
- Q2 pad 2: Net-(Q2-D) -> /PowerControl/BATT
- Q2 pad 3: /PowerControl/BATT -> Net-(Q2-D)
- Q4 pad 2: Net-(Q2-D) -> /PowerControl/BATT_UPPER
- Q4 pad 3: /PowerControl/BATT_UPPER -> Net-(Q2-D)
- Q5 pad 2: Net-(Q5-D) -> /PowerControl/GPU
- Q5 pad 3: /PowerControl/GPU -> Net-(Q5-D)
- Q7 pad 2: Net-(Q7-D) -> +VSW
- Q7 pad 3: Net-(D4-K) -> Net-(Q1-D)
Routing:
- net Net-(Q1-G): track 19.5 -> 25.5 mm
- net Net-(D4-K): track 44.3 -> 48.4 mm
- net Net-(Q5-G): track 19.0 -> 21.9 mm
- net +VSW: track 0.00 -> 2.54 mm
- net Net-(Q2-G): track 18.6 -> 16.5 mm
- net /PowerControl/BATT: track 0.00 -> 1.99 mm
- net LTC4353_EN2: track 47.1 -> 48.2 mm
- net Net-(Q3-D): track 3.72 -> 2.90 mm
- net GND: vias 225 -> 222
- added copper zone on F.Cu, net Net-(Q1-D)
- removed copper zone on F.Cu, net Net-(Q7-D)

Commit message: Build-4作成完了
Parts:
- removed the Q1 at (1.96, 1.90)
- added D10: SS2040FL, Diode_SMD:D_SOD-123F, B.Cu at (159.9, 115.0)
- J1, J2: value DF51-2P-2DS -> DF1B-2S-2.5R; footprint TSRP_Connector_Hirose:DF51-2P-2DS -> TSRP_Connector:DF1B-2S-2.5R
- moved J1 9.23 mm to (134.7, 74.6)
- moved J2 9.07 mm to (139.7, 125.4)
- moved C4 2.14 mm to (132.1, 80.4)
- moved R8 1.32 mm to (131.9, 83.2)
Routing:
- net +5VD: track 7.55 -> 14.5 mm, vias 0 -> 1
- net +12V: track 117.9 -> 120.5 mm, vias 2 -> 3
- net Net-(D4-K): track 48.4 -> 49.8 mm
- net GND: vias 222 -> 257

Commit message: Build-4発注済み
Other:
- board text added: "Power Module Build-4"
- board text removed: "Power Module Build-3"
Changed lines of the file:
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@@
 		)
 	)
-	(gr_text "Power Module  Build-3"
+	(gr_text "Power Module  Build-4"
 		(at 161.406 134.288 0)
 		(layer "B.SilkS")

Commit message: Build-5を作成
Parts:
- removed U7: MCP2515-xSO, Package_SO:TSSOP-20_4.4x6.5mm_P0.65mm
- added D11: SS2040FL, Diode_SMD:D_SOD-123F, F.Cu at (110.7, 86.2)
- added R23: 4.7kR, Resistor_SMD:R_0603_1608Metric_Pad0.98x0.95mm_HandSolder, F.Cu at (110.5, 112.6)
- added U2: MCP2515-xST, Package_SO:TSSOP-20_4.4x6.5mm_P0.65mm, F.Cu at (178.3, 116.1)
- C1: value 100uF -> 220uF
- C21: value 0.0056uF -> 0.056uF
- D3: value Orange -> Green
- D6: value SB34AFC -> SS2040FL; footprint Diode_SMD:D_SMA_Handsoldering -> Diode_SMD:D_SOD-123F
- moved D6 2.54 mm to (127.4, 86.1), turned to -90 degrees
- moved R24 1.37 mm to (172.0, 118.6)
- moved PS1 1.14 mm to (121.5, 81.9)
- moved C13 1.14 mm to (173.5, 120.4)
- moved C15 0.64 mm to (185.3, 121.2)
- moved C14 0.63 mm to (185.3, 107.2)
- moved Y1 0.63 mm to (186.4, 116.6)
Connections:
- U1 pad 14: +5V -> Net-(D11-K)
Routing:
- net +3.3V: track 145.4 -> 169.3 mm
- net +12V: track 120.5 -> 113.7 mm
- net +5V: track 12.2 -> 6.93 mm
- net Net-(D11-K): track 0.00 -> 4.58 mm
- net SPI_CS_MCP2515: track 72.9 -> 74.9 mm
- net Net-(D6-K): track 8.82 -> 6.99 mm
- net SPI_MISO: track 68.8 -> 70.3 mm
- net SPI_MOSI: track 71.6 -> 72.9 mm
- net SPI_SCK: track 65.4 -> 66.0 mm
- net Net-(U2-~{RESET}): track 3.24 -> 3.76 mm
- net GND: vias 257 -> 259
Other:
- board text added: "0x40"
- board text added: "0x41"
- board text added: "0x45"
- board text added: "Power Module Build-5"
- board text removed: "0b100 0000"
- board text removed: "0b100 0001"
- board text removed: "0b100 0101"
- board text removed: "Power Module Build-4"
