File: KiCAD/PowerControlModule/PowerControlModule.kicad_pcb (KiCad board)
At the start: 2 copper layers, 90 x 70 mm, 85 parts, among them J1 DF1B-2S-2.5R, J2 DF1B-2S-2.5R, J3 DF11-8DP-2DS, Q1 AO3401A, Q11 Si4162DY, Q12 Si4162DY, Q2 AO3401A, Q3 AO3400A, Q4 AO3401A, Q5 AO3401A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

Commit message: 修正した．発注する．
Parts:
- added R27: 10k, Resistor_SMD:R_0603_1608Metric, F.Cu at (126.9, 88.0)
- moved D6 5.08 mm to (127.3, 81.0)
- moved R21 0.51 mm to (169.4, 125.5)
- turned D3 to 90 degrees
Connections:
- D3 pad 1: Net-(D3-K) -> GND
- U1 pad 8: unconnected-(U1-GPIO1/RX-Pad8) -> LTC3119_PGOOD
- U11 pad 2: Net-(D3-K) -> LTC3119_PGOOD
Routing:
- net LTC3119_PGOOD: track 0.00 -> 67.0 mm, vias 0 -> 3
- net Net-(D3-K): track 42.7 -> 0.00 mm, vias 1 -> 0
- net +3.3V: track 169.3 -> 177.0 mm, vias 8 -> 10
- net +12V: track 113.7 -> 118.8 mm
- net Net-(D3-A): track 5.33 -> 2.02 mm
- net GND: vias 259 -> 263
