File: KiCAD/PowerControlModule/CanInterface.kicad_sch (KiCad schematic)
At the start: 12 parts, among them J3 DF11-8DP-2DS, U8 MCP2515-xSO, U9 MCP2562-E-SN, Y1 8MHz

Commit message: PowerControlModuleを作成．ソフトウェアの開発も進めなければいけない....
Parts:
- added C19, C20: 2.2uF, Capacitor_SMD:C_0603_1608Metric_Pad1.08x0.95mm_HandSolder, symbol Device:C_Small
- added U9: MCP1792x-5002xCB, Package_TO_SOT_SMD:SOT-23_Handsoldering, symbol Regulator_Linear:MCP1792x-5002xCB
- renumbered C15 to C13, C16 to C14, C17 to C15, C18 to C16, C19 to C17, D7 to D5, R20 to R24, R21 to R25, U8 to U7, U9 to U8
Connections:
- net +12V: now also C19.1, U9.3 (VI)
- net GND: now also C19.2, C20.2, U9.1 (GND)
- net +5V renamed +5VD
- net +5VD: now also C20.1, U9.2 (VO)
Other:
- moved on the sheet: C16, C17, D5, J3, R25, U8

Commit message: Build-3完成．本日発注．
Parts:
- D5: value GS1010FL -> SMAJ45A; footprint Diode_SMD:D_SOD-123 -> Diode_SMD:D_SMA
- R24: value 10K -> 10kR
- R25: value 120 -> 120R
- Y1: footprint Crystal:Crystal_SMD_HC49-SD -> Crystal:Crystal_HC49-4H_Vertical
Changed lines of the file:
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@@
+			)
+		)
+		(property "Sim.Type" ""
+			(at 59.69 36.83 0)
+			(effects
+				(font
+					(size 1.27 1.27)
+				)
 			)
 		)
@@
 			)
 		)
-		(property "Footprint" "Crystal:Crystal_SMD_HC49-SD"
+		(property "Footprint" "Crystal:Crystal_HC49-4H_Vertical"
 			(at 64.77 107.95 0)
 			(effects
@@
 			)
 		)
-		(property "Datasheet" "https://akizukidenshi.com/catalog/g/gP-08667/"
+		(property "Datasheet" "https://akizukidenshi.com/catalog/g/g108667/"
 			(at 64.77 107.95 0)
 			(effects
@@
 				)
 				(hide yes)
+			)
+		)
+		(property "Sim.Type" ""
+			(at 64.77 107.95 0)
+			(effects
+				(font
+					(size 1.27 1.27)
+				)
 			)
 		)
@@
 			)
 		)
+		(property "Sim.Type" ""
+			(at 129.54 38.1 0)
+			(effects
+				(font
+					(size 1.27 1.27)
+				)
+			)
+		)
 		(pin "2"
 		)
@@
 			)
 		)
+		(property "Sim.Type" ""
+			(at 69.85 114.3 0)
+			(effects
+				(font
+					(size 1.27 1.27)
+				)
+			)
+		)
 		(pin "1"
 		)
@@
 			)
 		)
-		(property "Value" "GS1010FL"
+		(property "Value" "SMAJ45A"
 			(at 138.43 134.6199 90)
 			(effects
@@
 			)
 		)
-		(property "Footprint" "Diode_SMD:D_SOD-123"
+		(property "Footprint" "Diode_SMD:D_SMA"
 			(at 135.89 133.35 0)
 			(effects
@@
 			)
 		)
-		(property "Datasheet" "https://akizukidenshi.com/catalog/g/g106014/"
+		(property "Datasheet" "https://akizukidenshi.com/catalog/g/g107409/"
 			(at 135.89 133.35 0)
 			(effects
@@
 				)
 				(hide yes)
+			)
+		)
+		(property "Sim.Type" ""
+			(at 135.89 133.35 0)
+			(effects
+				(font
+					(size 1.27 1.27)
+				)
 			)
 		)
@@
 			)
 		)
+		(property "Sim.Type" ""
+			(at 156.21 72.39 0)
+			(effects
+				(font
+					(size 1.27 1.27)
+				)
+			)
+		)
 		(pin "6"
 		)
@@
 			)
 		)
+		(property "Sim.Type" ""
+			(at 149.86 59.69 0)
+			(effects
+				(font
+					(size 1.27 1.27)
+				)
+			)
+		)
 		(pin "1"
 		)
@@
 			)
 		)
+		(property "Sim.Type" ""
+			(at 69.85 101.6 0)
+			(effects
+				(font
+					(size 1.27 1.27)
+				)
+			)
+		)
 		(pin "1"
 		)
@@
 				)
 				(hide yes)
+			)
+		)
+		(property "Sim.Type" ""
+			(at 116.84 121.92 0)
+			(effects
+				(font
+					(size 1.27 1.27)
+				)
 			)
 		)
@@
 			)
 		)
+		(property "Sim.Type" ""
+			(at 119.38 41.91 0)
+			(effects
+				(font
+					(size 1.27 1.27)
+				)
+			)
+		)
 		(pin "1"
 		)
@@
 			)
 		)
+		(property "Sim.Type" ""
+			(at 128.27 78.74 0)
+			(effects
+				(font
+					(size 1.27 1.27)
+				)
+			)
+		)
 		(pin "1"
 		)
@@
 			)
 		)
-		(property "Value" "120"
+		(property "Value" "120R"
 			(at 194.31 73.6599 0)
 			(effects
@@
 			)
 		)
+		(property "Sim.Type" ""
+			(at 191.77 72.39 0)
+			(effects
+				(font
+					(size 1.27 1.27)
+				)
+			)
+		)
 		(pin "2"
 		)
@@
 			)
 		)
+		(property "Sim.Type" ""
+			(at 63.5 66.04 0)
+			(effects
+				(font
+					(size 1.27 1.27)
+				)
+			)
+		)
 		(pin "15"
 		)
@@
 			)
 		)
-		(property "Value" "10K"
+		(property "Value" "10kR"
 			(at 85.09 77.47 90)
 			(effects
@@
 				)
 				(hide yes)
+			)
+		)
+		(property "Sim.Type" ""
+			(at 85.09 81.28 0)
+			(effects
+				(font
+					(size 1.27 1.27)
+				)
 			)
 		)
@@
 			)
 		)
+		(property "Sim.Type" ""
+			(at 143.51 41.91 0)
+			(effects
+				(font
+					(size 1.27 1.27)
+				)
+			)
+		)

Commit message: Build-4作成完了
Parts:
- added D10: SS2040FL, Diode_SMD:D_SOD-123F, symbol Device:D_Schottky
Connections:
- net +12V: now also D10.1 (K)
- net +5VD: now also D10.2 (A)
Other:
- moved on the sheet: C16, C17, C19, C20, D5, J3, R25, U8, U9

Commit message: Build-5を作成
Parts:
- removed U7: MCP2515-xSO, Package_SO:TSSOP-20_4.4x6.5mm_P0.65mm, symbol Interface_CAN_LIN:MCP2515-xSO
- added U2: MCP2515-xST, Package_SO:TSSOP-20_4.4x6.5mm_P0.65mm, symbol Interface_CAN_LIN:MCP2515-xST
Connections:
- net +3.3V: now also U2.20 (VDD)
- net CAN_RX: now also U2.2 (RXCAN)
- net CAN_TX: now also U2.1 (TXCAN)
- net GND: now also U2.10 (VSS)
- net OSC1: now also U2.9 (OSC1)
- net OSC2: now also U2.8 (OSC2)
- net SPI_CS_MCP2515: now also U2.18 (~{CS})
- net SPI_MISO: now also U2.17 (SO)
- net SPI_MOSI: now also U2.16 (SI)
- net SPI_SCK: now also U2.14 (SCK)
- net at R24.1: now also U2.19 (~{RESET})
Changed lines of the file:
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@@
 	)
 	(symbol
-		(lib_id "Interface_CAN_LIN:MCP2515-xSO")
+		(lib_id "Interface_CAN_LIN:MCP2515-xST")
 		(at 63.5 66.04 0)
 		(unit 1)
@@
 		(dnp no)
 		(fields_autoplaced yes)
-		(property "Reference" "U7"
+		(property "Reference" "U2"
 			(at 65.6433 43.18 0)
 			(effects
@@
 			)
 		)
-		(property "Value" "MCP2515-xSO"
+		(property "Value" "MCP2515-xST"
 			(at 65.6433 45.72 0)
 			(effects
@@
 			)
 		)
-		(property "Description" "Stand-Alone CAN Controller with SPI Interface, SOIC-18"
+		(property "Description" "Stand-Alone CAN Controller with SPI Interface, TSSOP-20"
 			(at 63.5 66.04 0)
 			(effects
@@
 			)
 		)
-		(property "Sim.Type" ""
-			(at 63.5 66.04 0)
-			(effects
-				(font
-					(size 1.27 1.27)
-				)
-			)
+		(pin "17"
+		)
+		(pin "20"
+		)
+		(pin "2"
+		)
+		(pin "16"
+		)
+		(pin "14"
+		)
+		(pin "8"
+		)
+		(pin "18"
+		)
+		(pin "3"
+		)
+		(pin "6"
 		)
 		(pin "15"
 		)
-		(pin "18"
-		)
 		(pin "9"
 		)
-		(pin "16"
-		)
-		(pin "8"
+		(pin "10"
 		)
 		(pin "13"
 		)
-		(pin "11"
+		(pin "5"
+		)
+		(pin "19"
 		)
 		(pin "7"
 		)
-		(pin "2"
+		(pin "11"
+		)
+		(pin "1"
+		)
+		(pin "12"
 		)
 		(pin "4"
 		)
-		(pin "6"
-		)
-		(pin "17"
-		)
-		(pin "3"
-		)
-		(pin "1"
-		)
-		(pin "5"
-		)
-		(pin "12"
-		)
-		(pin "10"
-		)
-		(pin "14"
-		)
 		(instances
-			(project "PowerControlModule"
+			(project ""
 				(path "/cd54ca1c-60d1-49a2-85aa-1c2ce8b76912/4bc17551-98e8-4384-b981-0ab382368ca6"
-					(reference "U7")
+					(reference "U2")
 					(unit 1)
 				)

Commit message: 修正した．発注する．
Parts:
- added D3: Green, LED_SMD:LED_0603_1608Metric_Pad1.05x0.95mm_HandSolder, symbol Device:LED_Small
- added R21: 3.6kR, Resistor_SMD:R_0603_1608Metric_Pad0.98x0.95mm_HandSolder, symbol Device:R_Small
Connections:
- net +12V: now also R21.1
- net GND: now also D3.1 (K)
- new net: D3.2 (A), R21.2
Other:
- moved on the sheet: D5
