File: KiCAD/SensingModule/Peripheral.kicad_sch (KiCad schematic)
At the start: 12 parts, among them J3 DF51-2P-2DS, J4 DF51A-4P-2DS, U5 MB85RQ8MX, U6 MB85RQ8MX, U7 MB85RQ8MX

Commit message: Build-2完成．発注．
Parts:
- removed C17: 0.1uF, Capacitor_SMD:C_0603_1608Metric_Pad1.08x0.95mm_HandSolder, symbol Device:C
- U2: value ~ -> BNO055
Connections:
- net I2C_SCK renamed I2C_SCL
Other:
- moved on the sheet: J3, R15, U14
