File: KiCAD/SensingModule/CanInterface.kicad_sch (KiCad schematic)
At the start: 14 parts, among them U3 MCP2562-E-P, U4 MCP2515-I/P, Y1 8MHz

Commit message: 配線をつなげようとしたがうまくいかず　もう少し考えてみる
Parts:
- U3: footprint Package_DIP:DIP-8_W7.62mm -> Package_SO:SOIC-8_3.9x4.9mm_P1.27mm
- U4: footprint Package_DIP:DIP-18_W7.62mm -> Package_SO:SOIC-18W_7.5x11.6mm_P1.27mm
Changed lines of the file:
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@@
 (kicad_sch
-	(version 20231120)
+	(version 20250114)
 	(generator "eeschema")
-	(generator_version "8.0")
+	(generator_version "9.0")
 	(paper "A4")
 	(junction
@@
 			)
 		)
-		(property "Footprint" "Package_DIP:DIP-18_W7.62mm"
+		(property "Footprint" "Package_SO:SOIC-18W_7.5x11.6mm_P1.27mm"
 			(at 199.39 59.69 0)
 			(effects
@@
 			)
 		)
-		(property "Footprint" "Package_DIP:DIP-8_W7.62mm"
+		(property "Footprint" "Package_SO:SOIC-8_3.9x4.9mm_P1.27mm"
 			(at 87.63 72.39 0)
 			(effects
@@
 			)
 		)
-		(property "Datasheet" "https://akizukidenshi.com/catalog/g/gI-14383/"
+		(property "Datasheet" "https://akizukidenshi.com/catalog/g/g114383/"
 			(at 87.63 59.69 0)
 			(effects

Commit message: きれいに配線できるようになった．
Parts:
- U4: footprint Package_SO:SOIC-18W_7.5x11.6mm_P1.27mm -> Package_SO:TSSOP-20_4.4x6.5mm_P0.65mm
Connections:
- net +3.3V renamed +3.3VP
Other:
- moved on the sheet: C6, C7, C8, R14, U4, Y1

Commit message: Build-2完成．発注．
Parts:
- D5, D6: value B -> Blue
Other:
- moved on the sheet: C7, C8, D5, D6, R12, R13, Y1

Commit message: Build-3を作成
Parts:
- removed U3: MCP2562-E-P, Package_SO:SOIC-8_3.9x4.9mm_P1.27mm, symbol Interface_CAN_LIN:MCP2562-E-P
- removed U4: MCP2515-I/P, Package_SO:TSSOP-20_4.4x6.5mm_P0.65mm, symbol MCP2515-I_P:MCP2515-I/P
- added U4: MCP2515-xST, Package_SO:TSSOP-20_4.4x6.5mm_P0.65mm, symbol Interface_CAN_LIN:MCP2515-xST
- added U9: MCP2562-E-SN, Package_SO:SOIC-8_3.9x4.9mm_P1.27mm, symbol Interface_CAN_LIN:MCP2562-E-SN
- Y1: footprint Crystal:Crystal_SMD_HC49-SD -> Crystal:Crystal_HC49-4H_Vertical
Connections:
- net +3.3VP: now also R14.2, U4.20 (VDD), U9.5 (Vio); no longer R14.1
- net +5V: now also U9.3 (VDD)
- net CAN_H: now also U9.7 (CANH)
- net CAN_L: now also U9.6 (CANL)
- net CAN_RX: now also U4.2 (RXCAN), U9.4 (RXD)
- net CAN_TX: now also U4.1 (TXCAN), U9.1 (TXD)
- net GND: now also U4.10 (VSS), U9.2 (VSS), U9.8 (STBY)
- net OSC1: now also U4.9 (OSC1)
- net OSC2: now also U4.8 (OSC2)
- net SPI_CS_MCP: now also U4.18 (~{CS})
- net SPI_MISO: now also U4.17 (SO)
- net SPI_MOSI: now also U4.16 (SI)
- net SPI_SCLK: now also U4.14 (SCK)
- new net: R14.1, U4.19 (~{RESET})
Other:
- moved on the sheet: C6, C7, C8, R14, Y1
