File: KiCAD/SensingModule/Power.kicad_sch (KiCad schematic)
At the start: 8 parts, among them U8 RT9080-33GJ5

Commit message: 修正した．発注する．
Parts:
- D7: value SB34AFC -> SS2040FL; footprint Diode_SMD:D_SMA_Handsoldering -> Diode_SMD:D_SOD-123F
Changed lines of the file:
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@@
 			)
 		)
-		(property "Value" "SB34AFC"
+		(property "Value" "SS2040FL"
 			(at 77.7875 45.72 0)
 			(effects
@@
 			)
 		)
-		(property "Footprint" "Diode_SMD:D_SMA_Handsoldering"
+		(property "Footprint" "Diode_SMD:D_SOD-123F"
 			(at 77.47 49.53 0)
 			(effects
@@
 			)
 		)
-		(property "Datasheet" "https://akizukidenshi.com/catalog/g/g117502/"
+		(property "Datasheet" "https://akizukidenshi.com/catalog/g/g102073/"
 			(at 77.47 49.53 0)
 			(effects
