File: KiCAD/ValveControlModule/Periferal.kicad_sch (KiCad schematic)
At the start: 15 parts, among them J3 DF51A-4P-2DS, U6 MB85RQ8MX, U7 MB85RQ8MX, U8 TC7S14F, U9 TC7S14F

Commit message: Build-2完成．発注．
Parts:
- removed C19: 0.1uF, Capacitor_SMD:C_0603_1608Metric_Pad1.08x0.95mm_HandSolder, symbol Device:C
- removed U7: MB85RQ8MX, Package_SO:SOIC-16W_7.5x10.3mm_P1.27mm, symbol TSRP_IC:MB85RQ8MX
