File: KiCAD/THRValveControlModule/THRValveControlModule.kicad_pcb (KiCad board)
At the start: 2 copper layers, 99 x 75 mm, 54 parts, among them J1 B4B-XH-A(LF)(SN), J2 B3B-XH-A(LF)(SN), J3 B3B-XH-A(LF)(SN), J4 XT30PW-M, J5 DF51A-4P-2DSA, J6 SSD1306, J7 DF51A-8DP-2DS, Q1 IRLML6344TRPBFTR, U1 XIAO-RA4M1-SMD, U10 MB85RQ8MX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

Commit message: 基板発注完了
Parts:
- moved G*** 0.18 mm to (113.5, 78.9)
