File: KiCAD/THRValveControlModule/motorInterface.kicad_sch (KiCad schematic)
At the start: 7 parts, among them J1 B4B-XH-A(LF)(SN), J2 B3B-XH-A(LF)(SN), J3 B3B-XH-A(LF)(SN), U5 MAX485E

Commit message: 基板発注完了
Parts:
- D2: Supplyer (none) -> https://akizukidenshi.com/catalog/g/g129635/
Changed lines of the file:
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@@
+			)
+		)
+		(property "Supplyer" "https://akizukidenshi.com/catalog/g/g129635/"
+			(at 118.11 77.47 90)
+			(effects
+				(font
+					(size 1.27 1.27)
+				)
+				(hide yes)
 			)
 		)
