File: KiCAD/THRValveControlModule/periferal.kicad_sch (KiCad schematic)
At the start: 21 parts, among them J5 DF51A-4P-2DSA, J6 SSD1306, Q1 IRLML6344TRPBFTR, SW2 SKRPACE010, U10 MB85RQ8MX, U8 TC7S14F, U9 TC7S14F

Commit message: 基板発注完了
Parts:
- C18: Supplyer (none) -> https://akizukidenshi.com/catalog/g/g113374/
Changed lines of the file:
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@@
 			)
 		)
-		(property "Datasheet" "~"
+		(property "Datasheet" "https://www.hirose.com/ja/product/p/CL0543-5107-0-00"
 			(at 30.48 86.36 0)
 			(effects
@@
 			)
 		)
-		(property "Datasheet" ""
+		(property "Datasheet" "https://www.ramxeed.com/jp/home/wp-content/uploads/2024/12/MB85RQ8MX-DS1v1-J.pdf"
 			(at 162.56 119.126 0)
 			(effects
@@
 			)
 		)
-		(property "Datasheet" "~"
+		(property "Datasheet" "https://akizukidenshi.com/goodsaffix/UGCT7525AN4.pdf"
 			(at 84.836 121.92 0)
 			(effects
@@
 			(at 168.91 106.68 0)
 			(effects
+				(font
+					(size 1.27 1.27)
+				)
+				(hide yes)
+			)
+		)
+		(property "Supplyer" "https://akizukidenshi.com/catalog/g/g113374/"
+			(at 168.91 106.68 0)
+			(effects
